File: 01_hardware/kicad_project/can.kicad_sch (KiCad schematic)
At the start: 15 parts, among them J3 CAN A, J4 CAN B, U9 CA-IS3062VW

Commit message: add CAN termination res jumper
Parts:
- removed JP1: TERM, Connector_PinHeader_2.54mm:PinHeader_1x02_P2.54mm_Vertical, symbol Connector_Generic:Conn_01x02
- added JP1: TERM, Connector_PinHeader_2.54mm:PinHeader_2x02_P2.54mm_Vertical, symbol Connector_Generic:Conn_02x02_Odd_Even
Connections:
- net CANH: now also JP1.2 (Pin_2); no longer R30.1
- net CANL: now also JP1.3 (Pin_3)
- net CAN_TL: now also JP1.4 (Pin_4)
- new net CAN_TH: JP1.1 (Pin_1), R30.1
Changed lines of the file:
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@@
     (comment 2 "Sheet 8: Isolated CAN")
   )
-  (junction (at 205.74 99.06) (diameter 0) (color 0 0 0 0)
-  )
-  (junction (at 210.82 101.6) (diameter 0) (color 0 0 0 0)
-  )
   (junction (at 210.82 115.57) (diameter 0) (color 0 0 0 0)
   )
-  (junction (at 238.76 101.6) (diameter 0) (color 0 0 0 0)
+  (junction (at 238.76 96.52) (diameter 0) (color 0 0 0 0)
   )
   (junction (at 243.84 99.06) (diameter 0) (color 0 0 0 0)
@@
     (stroke (width 0) (type default))
   )
-  (wire (pts (xy 210.82 102.87) (xy 210.82 101.6))
-    (stroke (width 0) (type default))
-  )
-  (wire (pts (xy 210.82 101.6) (xy 210.82 100.33))
+  (wire (pts (xy 210.82 102.87) (xy 210.82 100.33))
     (stroke (width 0) (type default))
   )
@@
     (stroke (width 0) (type default))
   )
-  (wire (pts (xy 203.2 128.27) (xy 205.74 128.27))
-    (stroke (width 0) (type default))
-  )
-  (wire (pts (xy 203.2 125.73) (xy 205.74 125.73))
+  (wire (pts (xy 190.5 114.3) (xy 187.96 114.3))
+    (stroke (width 0) (type default))
+  )
+  (wire (pts (xy 203.2 114.3) (xy 205.74 114.3))
+    (stroke (width 0) (type default))
+  )
+  (wire (pts (xy 190.5 116.84) (xy 187.96 116.84))
+    (stroke (width 0) (type default))
+  )
+  (wire (pts (xy 203.2 116.84) (xy 205.74 116.84))
     (stroke (width 0) (type default))
   )
@@
     (stroke (width 0) (type default))
   )
-  (wire (pts (xy 205.74 128.27) (xy 210.82 128.27))
+  (wire (pts (xy 210.82 100.33) (xy 187.96 100.33))
+    (stroke (width 0) (type default))
+  )
+  (wire (pts (xy 187.96 100.33) (xy 187.96 114.3))
+    (stroke (width 0) (type default))
+  )
+  (wire (pts (xy 210.82 128.27) (xy 205.74 128.27))
+    (stroke (width 0) (type default))
+  )
+  (wire (pts (xy 205.74 128.27) (xy 205.74 116.84))
+    (stroke (width 0) (type default))
+  )
+  (wire (pts (xy 238.76 101.6) (xy 238.76 96.52))
+    (stroke (width 0) (type default))
+  )
+  (wire (pts (xy 238.76 96.52) (xy 166.37 96.52))
+    (stroke (width 0) (type default))
+  )
+  (wire (pts (xy 292.1 96.52) (xy 238.76 96.52))
+    (stroke (width 0) (type default))
+  )
+  (wire (pts (xy 243.84 101.6) (xy 243.84 99.06))
+    (stroke (width 0) (type default))
+  )
+  (wire (pts (xy 243.84 99.06) (xy 166.37 99.06))
+    (stroke (width 0) (type default))
+  )
+  (wire (pts (xy 292.1 99.06) (xy 243.84 99.06))
     (stroke (width 0) (type default))
   )
@@
     (stroke (width 0) (type default))
   )
-  (wire (pts (xy 210.82 100.33) (xy 210.82 96.52))
-    (stroke (width 0) (type default))
-  )
-  (wire (pts (xy 210.82 96.52) (xy 166.37 96.52))
-    (stroke (width 0) (type default))
-  )
-  (wire (pts (xy 238.76 101.6) (xy 210.82 101.6))
-    (stroke (width 0) (type default))
-  )
-  (wire (pts (xy 292.1 96.52) (xy 238.76 96.52))
-    (stroke (width 0) (type default))
-  )
-  (wire (pts (xy 238.76 96.52) (xy 238.76 101.6))
-    (stroke (width 0) (type default))
-  )
-  (wire (pts (xy 205.74 125.73) (xy 205.74 101.6))
-    (stroke (width 0) (type default))
-  )
-  (wire (pts (xy 205.74 101.6) (xy 205.74 99.06))
-    (stroke (width 0) (type default))
-  )
-  (wire (pts (xy 205.74 99.06) (xy 166.37 99.06))
-    (stroke (width 0) (type default))
-  )
-  (wire (pts (xy 243.84 101.6) (xy 243.84 99.06))
-    (stroke (width 0) (type default))
-  )
-  (wire (pts (xy 243.84 99.06) (xy 205.74 99.06))
-    (stroke (width 0) (type default))
-  )
-  (wire (pts (xy 292.1 99.06) (xy 243.84 99.06))
-    (stroke (width 0) (type default))
+  (label "CAN_TH" (at 187.96 114.3 180)
+    (effects (font (size 1.0 1.0)) (justify right bottom))
   )
   (label "CAN_TL" (at 210.82 128.27 270)
     (effects (font (size 1.0 1.0)) (justify right bottom))
   )
+  (label "CANH" (at 166.37 96.52 0)
+    (effects (font (size 1.0 1.0)) (justify left bottom))
+  )
+  (label "CANL" (at 166.37 99.06 0)
+    (effects (font (size 1.0 1.0)) (justify left bottom))
+  )
   (label "CAN_MID" (at 220.98 115.57 90)
     (effects (font (size 1.0 1.0)) (justify left bottom))
   )
-  (label "CANH" (at 166.37 96.52 0)
+  (label "CANH" (at 205.74 114.3 0)
     (effects (font (size 1.0 1.0)) (justify left bottom))
   )
-  (label "CANL" (at 205.74 125.73 0)
-    (effects (font (size 1.0 1.0)) (justify left bottom))
+  (label "CANL" (at 187.96 116.84 180)
+    (effects (font (size 1.0 1.0)) (justify right bottom))
   )
   (label "CANH" (at 292.1 111.76 180)
@@
     (pin "2")
   )
-  (symbol (lib_id "Connector_Generic:Conn_01x02") (at 198.12 128.27 180) (unit 1)
-    (in_bom yes) (on_board yes)
-    (property "Reference" "JP1" (id 0) (at 198.12 122.844 0)
-      (effects (font (size 1.27 1.27)))
-    )
-    (property "Value" "TERM" (id 1) (at 198.12 131.156 0)
-      (effects (font (size 1.27 1.27)))
-    )
-    (property "Footprint" "Connector_PinHeader_2.54mm:PinHeader_1x02_P2.54mm_Vertical" (id 2) (at 198.12 128.27 0)
-      (effects (font (size 1.27 1.27)) hide)
-    )
-    (property "Datasheet" "" (id 3) (at 198.12 128.27 0)
-      (effects (font (size 1.27 1.27)) hide)
-    )
-    (property "LCSC" "" (id 4) (at 198.12 128.27 0)
-      (effects (font (size 1.27 1.27)) hide)
-    )
-    (property "MPN" "TERM" (id 5) (at 198.12 128.27 0)
-      (effects (font (size 1.27 1.27)) hide)
-    )
-    (pin "1")
-    (pin "2")
+  (symbol (lib_id "Connector_Generic:Conn_02x02_Odd_Even") (at 195.58 114.3 0) (unit 1)
+    (in_bom yes) (on_board yes)
+    (property "Reference" "JP1" (id 0) (at 196.85 111.414 0)
+      (effects (font (size 1.27 1.27)))
+    )
+    (property "Value" "TERM" (id 1) (at 196.85 119.726 0)
+      (effects (font (size 1.27 1.27)))
+    )
+    (property "Footprint" "Connector_PinHeader_2.54mm:PinHeader_2x02_P2.54mm_Vertical" (id 2) (at 195.58 114.3 0)
+      (effects (font (size 1.27 1.27)) hide)
+    )
+    (property "Datasheet" "" (id 3) (at 195.58 114.3 0)
+      (effects (font (size 1.27 1.27)) hide)
+    )
+    (property "LCSC" "" (id 4) (at 195.58 114.3 0)
+      (effects (font (size 1.27 1.27)) hide)
+    )
+    (property "MPN" "TERM" (id 5) (at 195.58 114.3 0)
+      (effects (font (size 1.27 1.27)) hide)
+    )
+    (pin "1")
+    (pin "2")
+    (pin "3")
+    (pin "4")
   )
   (symbol (lib_id "Power_Protection:NUP2105L") (at 241.3 109.22 0) (unit 1)
