File: 01_hardware/kicad_project/can.kicad_sch (KiCad schematic)
At the start: 15 parts, among them J3 CAN A, J4 CAN B, U9 CA-IS3062VW

Commit message: Rev D order prep: common F1/L2/L3 parts, JLC-checked LCSC numbers, assembly files
- F1: 2512 -> 1206 7 A 63 V fuse (Littelfuse 0458007.DR, C206980; 2nd source Schurter 3413.0326.11)
- L2/L3: SRP5030 -> 5040 shielded 47 uH (SWPA5040S470MT, C86617; 2nd source SRN5040-470M, NRS5040T470MMGK)
- EN_AUX re-routed off the L2 pad gap; VIN track centred between the L3 pads (0.4 mm each side)
- LCSC numbers checked in the JLCPCB library for every assembled part (design.py JLC_LCSC),
  written to the BOMs, schematic and PCB fields
- New JLC assembly upload files DCDC_JLC_BOM.csv / DCDC_JLC_CPL.csv (217 parts; U1, T1,
  connectors, headers and SW1 hand-soldered) and jlc_order_files.py to rebuild them
- 03_calculations/aux_fuse_check.py: aux inductor peak 0.27 A vs 1.1 A Isat; F1 4.8 A at 12 V / 50 W
- Design notes (docx/pdf), README, Gerbers, CPL, PDFs and DRC report regenerated
- Checks: DRC (JLC rules) 0 errors / 0 unconnected, netlist 134 nets / 257 parts 0 errors,
  isolation check 0 errors, silkscreen clean

Co-Authored-By: Claude Opus 5.5 <noreply@anthropic.com>
Claude-Session: https://claude.ai/code/session_01A35wrnwFKLPSaRSxxHs471
Parts:
- C49, C52: LCSC (none) -> C15850
- C50, C53, C54: LCSC (none) -> C1525
- C51: LCSC (none) -> C52923
- C55: LCSC (none) -> C53987
- D3: LCSC (none) -> C14486
- R30, R31: LCSC (none) -> C2933247
Changed lines of the file:
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@@
       (effects (font (size 1.27 1.27)) hide)
     )
-    (property "LCSC" "" (id 4) (at 96.52 76.2 0)
+    (property "LCSC" "C15850" (id 4) (at 96.52 76.2 0)
       (effects (font (size 1.27 1.27)) hide)
     )
@@
       (effects (font (size 1.27 1.27)) hide)
     )
-    (property "LCSC" "" (id 4) (at 109.22 76.2 0)
+    (property "LCSC" "C1525" (id 4) (at 109.22 76.2 0)
       (effects (font (size 1.27 1.27)) hide)
     )
@@
       (effects (font (size 1.27 1.27)) hide)
     )
-    (property "LCSC" "" (id 4) (at 121.92 76.2 0)
+    (property "LCSC" "C52923" (id 4) (at 121.92 76.2 0)
       (effects (font (size 1.27 1.27)) hide)
     )
@@
       (effects (font (size 1.27 1.27)) hide)
     )
-    (property "LCSC" "" (id 4) (at 182.88 73.66 0)
+    (property "LCSC" "C15850" (id 4) (at 182.88 73.66 0)
       (effects (font (size 1.27 1.27)) hide)
     )
@@
       (effects (font (size 1.27 1.27)) hide)
     )
-    (property "LCSC" "" (id 4) (at 195.58 73.66 0)
+    (property "LCSC" "C1525" (id 4) (at 195.58 73.66 0)
       (effects (font (size 1.27 1.27)) hide)
     )
@@
       (effects (font (size 1.27 1.27)) hide)
     )
-    (property "LCSC" "" (id 4) (at 208.28 73.66 0)
+    (property "LCSC" "C1525" (id 4) (at 208.28 73.66 0)
       (effects (font (size 1.27 1.27)) hide)
     )
@@
       (effects (font (size 1.27 1.27)) hide)
     )
-    (property "LCSC" "" (id 4) (at 210.82 106.68 0)
+    (property "LCSC" "C2933247" (id 4) (at 210.82 106.68 0)
       (effects (font (size 1.27 1.27)) hide)
     )
@@
       (effects (font (size 1.27 1.27)) hide)
     )
-    (property "LCSC" "" (id 4) (at 210.82 121.92 0)
+    (property "LCSC" "C2933247" (id 4) (at 210.82 121.92 0)
       (effects (font (size 1.27 1.27)) hide)
     )
@@
       (effects (font (size 1.27 1.27)) hide)
     )
-    (property "LCSC" "" (id 4) (at 220.98 121.92 0)
+    (property "LCSC" "C53987" (id 4) (at 220.98 121.92 0)
       (effects (font (size 1.27 1.27)) hide)
     )
@@
       (effects (font (size 1.27 1.27)) hide)
     )
-    (property "LCSC" "" (id 4) (at 241.3 109.22 0)
-      (effects (font (size 1.27 1.27)) hide)
-    )
+    (property "LCSC" "C14486" (id 4) (at 241.3 109.22 0)
+      (effects (font (size 1.27 1.27)) hide)
+    )

Commit message: Rev E BOM: in-stock LCSC first source for every part; 2nd/3rd sources checked
- First sources swapped (same footprints, layout unchanged): U1 STM32G474RBT3,
  Q2/Q3/Q5/Q6 NCEP068N10G, 10k 0402 FOJAN, 100n 0402 merged onto C307331,
  1u 0402 CCTC, R62/R63/R89/R82, FB1 Murata BLM18KG601SN1D, L2/L3 cjiang
  FNR5040S470MT, C82 KEMET C0G (was X7R), RS1 Milliohm HoJLR2512, SS110 MDD
- LCSC part numbers for the hand-soldered headers (J1-J5, J7, JP1)
- Schematic and PCB fields, BOM, JLC BOM/CPL, PDFs and design notes regenerated;
  netlist check 0 errors, DRC unchanged
- BOM_sourcing_revE.xlsx: live LCSC stock 2026-10-20, 2nd/3rd sources checked
  for pinout / land pattern / ratings, PCB reserve options for T2 and U9

Co-Authored-By: Claude Opus 5.5 <noreply@anthropic.com>
Claude-Session: https://claude.ai/code/session_01A35wrnwFKLPSaRSxxHs471
Parts:
- C50, C53, C54: LCSC C1525 -> C307331
- C51: LCSC C52923 -> C20539426
- J3, J4: LCSC (none) -> C42419910; MPN 2.54 mm 1x3 male pin header -> PZ254V-11-03P-A40
- JP1: LCSC (none) -> C45384660; MPN TERM -> PZ254V-12-04P-A40
Changed lines of the file:
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@@
       (effects (font (size 1.27 1.27)) hide)
     )
-    (property "LCSC" "C1525" (id 4) (at 109.22 76.2 0)
+    (property "LCSC" "C307331" (id 4) (at 109.22 76.2 0)
       (effects (font (size 1.27 1.27)) hide)
     )
@@
       (effects (font (size 1.27 1.27)) hide)
     )
-    (property "LCSC" "C52923" (id 4) (at 121.92 76.2 0)
+    (property "LCSC" "C20539426" (id 4) (at 121.92 76.2 0)
       (effects (font (size 1.27 1.27)) hide)
     )
@@
       (effects (font (size 1.27 1.27)) hide)
     )
-    (property "LCSC" "C1525" (id 4) (at 195.58 73.66 0)
+    (property "LCSC" "C307331" (id 4) (at 195.58 73.66 0)
       (effects (font (size 1.27 1.27)) hide)
     )
@@
       (effects (font (size 1.27 1.27)) hide)
     )
-    (property "LCSC" "C1525" (id 4) (at 208.28 73.66 0)
+    (property "LCSC" "C307331" (id 4) (at 208.28 73.66 0)
       (effects (font (size 1.27 1.27)) hide)
     )
@@
       (effects (font (size 1.27 1.27)) hide)
     )
-    (property "LCSC" "" (id 4) (at 195.58 114.3 0)
-      (effects (font (size 1.27 1.27)) hide)
-    )
-    (property "MPN" "TERM" (id 5) (at 195.58 114.3 0)
+    (property "LCSC" "C45384660" (id 4) (at 195.58 114.3 0)
+      (effects (font (size 1.27 1.27)) hide)
+    )
+    (property "MPN" "PZ254V-12-04P-A40" (id 5) (at 195.58 114.3 0)
       (effects (font (size 1.27 1.27)) hide)
     )
@@
       (effects (font (size 1.27 1.27)) hide)
     )
-    (property "LCSC" "" (id 4) (at 299.72 99.06 0)
-      (effects (font (size 1.27 1.27)) hide)
-    )
-    (property "MPN" "2.54 mm 1x3 male pin header" (id 5) (at 299.72 99.06 0)
+    (property "LCSC" "C42419910" (id 4) (at 299.72 99.06 0)
+      (effects (font (size 1.27 1.27)) hide)
+    )
+    (property "MPN" "PZ254V-11-03P-A40" (id 5) (at 299.72 99.06 0)
       (effects (font (size 1.27 1.27)) hide)
     )
@@
       (effects (font (size 1.27 1.27)) hide)
     )
-    (property "LCSC" "" (id 4) (at 299.72 114.3 0)
-      (effects (font (size 1.27 1.27)) hide)
-    )
-    (property "MPN" "2.54 mm 1x3 male pin header" (id 5) (at 299.72 114.3 0)
-      (effects (font (size 1.27 1.27)) hide)
-    )
+    (property "LCSC" "C42419910" (id 4) (at 299.72 114.3 0)
+      (effects (font (size 1.27 1.27)) hide)
+    )
+    (property "MPN" "PZ254V-11-03P-A40" (id 5) (at 299.72 114.3 0)
+      (effects (font (size 1.27 1.27)) hide)
+    )
