File: 01_hardware/kicad_project/mcu.kicad_sch (KiCad schematic)
At the start: 14 parts, among them U1 STM32G474RBT6, Y1 8MHz 12pF

Commit message: update D
Parts:
- added R100, R101, R102, R103, R104, R105, R90, R91, R92, R93, R94, R95, R96, R97, R98, R99: 10k, Resistor_SMD:R_0402_1005Metric, symbol Device:R
- added TP15: VIN_OVP, TestPoint:TestPoint_Pad_D1.5mm, symbol Connector:TestPoint
- C38, C39: value 18p C0G -> 12p C0G; MPN 18p C0G -> 12p C0G
- Y1: value 8MHz 12pF -> 16MHz 9pF; LCSC (none) -> C13738; MPN 8MHz 12pF -> X322516MLB4SI
Connections:
- net GND: now also R100.2, R101.2, R102.2, R103.2, R104.2, R105.2, R90.2, R91.2, R92.2, R93.2, R94.2, R95.2, R96.2, R97.2, R98.2, R99.2
- net NTC_SNS: now also U1.20 (PA6); no longer U1.18 (PA4)
- net SP_PA2: now reaches U1.14 (PA2)
- net SP_PA2: now also R93.1
- net SP_PA3: now reaches U1.17 (PA3)
- net SP_PA3: now also R94.1
- net SP_PC13: now reaches U1.2 (PC13)
- net SP_PC13: now also R90.1
- net SP_PA7: now reaches U1.21 (PA7)
- net SP_PA7: now also R96.1
- net SP_PB2: now reaches U1.26 (PB2)
- net SP_PB2: now also R97.1
- net SP_PC14: now reaches U1.3 (PC14)
- net SP_PC14: now also R91.1
- net SP_PB10: now reaches U1.30 (PB10)
- net SP_PB10: now also R98.1
- net SP_PC6: now reaches U1.38 (PC6)
- net SP_PC6: now also R99.1
- net SP_PC7: now reaches U1.39 (PC7)
- net SP_PC7: now also R100.1
- net SP_PC15: now reaches U1.4 (PC15)
- net SP_PC15: now also R92.1
- net SP_PA10: now reaches U1.44 (PA10)
- net SP_PA10: now also R101.1
- net VIN_OVP: now reaches U1.51 (PA15)
- net VIN_OVP: now also TP15.1
- net SP_PC12: now reaches U1.54 (PC12)
- net SP_PC12: now also R102.1
- net SP_PD2: now reaches U1.55 (PD2)
- net SP_PD2: now also R103.1
- net SP_PB4: now reaches U1.57 (PB4)
- net SP_PB4: now also R104.1
- net SP_PB5: now reaches U1.58 (PB5)
- net SP_PB5: now also R105.1
- new net SP_PA4: R95.1, U1.18 (PA4)
- no-connect marks 17 -> 0
Other:
- note added: "Unused GPIOs (PC13-15, PA2-4, PA7, PA10, PB2, PB4, PB5, PB10, PC6, PC7, PC12, PD2): 10k pull-down to GND each (R90-R105). PA4 is kept free for DAC1_OUT1 (Test_pin_DAC)."
