File: 01_hardware/kicad_project/mcu.kicad_sch (KiCad schematic)
At the start: 33 parts, among them U1 STM32G474RBT6, U19 REF3030AIDBZR, Y1 16MHz 9pF

Commit message: Rev E: isolated flyback aux supply, VREF+ back to 3.3 V, 1 oz re-layout
- New isolated aux flyback (sheet iso_pwr): UC3843B U20 from +10V_P, FDN86246 Q11,
  PA3855.006NLT EP13 T2, SS110 D9 -> isolated +10 V; secondary regulation TL431 U22 +
  EL357N opto U21 into COMP; RCD clamp D8/R116/C94; 2 A primary limit (R114)
- Secondary rails from the flyback, not VBUS: +10 V -> U4 10->5 V -> U5 TLV75533 3.3 V;
  MCU, CAN and drivers up before the LLC starts
- U12 -> CA-IS3742LW (data only); REF3030 U19 removed, VREF+ = +3V3A (3.3 V full scale)
- PCB re-placed / re-routed for 1 oz outer / 0.5 oz inner: power pours on F.Cu, In1 solid
  ground planes, gate loops as tight HO/HS pairs, 1.7 mm power-via pitch, per-pad GND vias
  in the MCU area; copper loss ~0.5 W at 50 W (03_calculations/copper_check.txt)
- DRC (JLC rules) 0 errors / 0 unconnected; netlist 148 nets / 284 parts 0 errors;
  isolation bands clear; BOM / JLC BOM+CPL / Gerbers / PDFs / design notes / READMEs updated
- Scripts: 04_scripts/pcb5 (placement, pours, routing, floods, island vias, silk),
  03_calculations/flyback_aux.py, copper_check.py

Co-Authored-By: Claude Opus 5.5 <noreply@anthropic.com>
Claude-Session: https://claude.ai/code/session_01A35wrnwFKLPSaRSxxHs471
Parts:
- removed C85: 1u 10V, Capacitor_SMD:C_0402_1005Metric, symbol Device:C
- removed U19: REF3030AIDBZR, Package_TO_SOT_SMD:SOT-23, symbol Reference_Voltage:REF3030
- R105: LCSC (none) -> C25744
Connections:
- net VREF_ADC is gone; now on net +3V3A: C36.1, C37.1, U1.28 (VREF+)

Commit message: Rev E BOM: in-stock LCSC first source for every part; 2nd/3rd sources checked
- First sources swapped (same footprints, layout unchanged): U1 STM32G474RBT3,
  Q2/Q3/Q5/Q6 NCEP068N10G, 10k 0402 FOJAN, 100n 0402 merged onto C307331,
  1u 0402 CCTC, R62/R63/R89/R82, FB1 Murata BLM18KG601SN1D, L2/L3 cjiang
  FNR5040S470MT, C82 KEMET C0G (was X7R), RS1 Milliohm HoJLR2512, SS110 MDD
- LCSC part numbers for the hand-soldered headers (J1-J5, J7, JP1)
- Schematic and PCB fields, BOM, JLC BOM/CPL, PDFs and design notes regenerated;
  netlist check 0 errors, DRC unchanged
- BOM_sourcing_revE.xlsx: live LCSC stock 2026-10-20, 2nd/3rd sources checked
  for pinout / land pattern / ratings, PCB reserve options for T2 and U9

Co-Authored-By: Claude Opus 5.5 <noreply@anthropic.com>
Claude-Session: https://claude.ai/code/session_01A35wrnwFKLPSaRSxxHs471
Parts:
- C30, C31, C32, C33, C34, C37, C40: LCSC C1525 -> C307331
- C36: LCSC C52923 -> C20539426
- R100, R101, R102, R103, R104, R105, R20, R90, R91, R92, R93, R94, R95, R96, R97, R98, R99: LCSC C25744 -> C2906861
- U1: value STM32G474RBT6 -> STM32G474RBT3; LCSC C529413 -> C1235414; MPN STM32G474RBT6 -> STM32G474RBT3
Other:
- title: STM32G474RBT6 MCU -> STM32G474RBT3 MCU
Changed lines of the file:
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@@
   (paper "A3")
   (title_block
-    (title "STM32G474RBT6 MCU")
+    (title "STM32G474RBT3 MCU")
     (date "2026-10-19")
     (rev "E")
     (comment 1 "DCDC LLC + 4SBB, 12-48 V in, 1.5-48 V / 5 A out, STM32G474")
-    (comment 2 "Sheet 7: STM32G474RBT6 MCU")
+    (comment 2 "Sheet 7: STM32G474RBT3 MCU")
   )
   (junction (at 143.51 96.52) (diameter 0) (color 0 0 0 0)
@@
       (effects (font (size 1.27 1.27)))
     )
-    (property "Value" "STM32G474RBT6" (id 1) (at 195.705 191.608 0)
+    (property "Value" "STM32G474RBT3" (id 1) (at 195.705 191.608 0)
       (effects (font (size 1.27 1.27)))
     )
@@
       (effects (font (size 1.27 1.27)) hide)
     )
-    (property "LCSC" "C529413" (id 4) (at 203.2 144.78 0)
-      (effects (font (size 1.27 1.27)) hide)
-    )
-    (property "MPN" "STM32G474RBT6" (id 5) (at 203.2 144.78 0)
+    (property "LCSC" "C1235414" (id 4) (at 203.2 144.78 0)
+      (effects (font (size 1.27 1.27)) hide)
+    )
+    (property "MPN" "STM32G474RBT3" (id 5) (at 203.2 144.78 0)
       (effects (font (size 1.27 1.27)) hide)
     )
@@
       (effects (font (size 1.27 1.27)) hide)
     )
-    (property "LCSC" "C1525" (id 4) (at 129.54 63.5 0)
+    (property "LCSC" "C307331" (id 4) (at 129.54 63.5 0)
       (effects (font (size 1.27 1.27)) hide)
     )
@@
       (effects (font (size 1.27 1.27)) hide)
     )
-    (property "LCSC" "C1525" (id 4) (at 142.24 63.5 0)
+    (property "LCSC" "C307331" (id 4) (at 142.24 63.5 0)
       (effects (font (size 1.27 1.27)) hide)
     )
@@
       (effects (font (size 1.27 1.27)) hide)
     )
-    (property "LCSC" "C1525" (id 4) (at 154.94 63.5 0)
+    (property "LCSC" "C307331" (id 4) (at 154.94 63.5 0)
       (effects (font (size 1.27 1.27)) hide)
     )
@@
       (effects (font (size 1.27 1.27)) hide)
     )
-    (property "LCSC" "C1525" (id 4) (at 167.64 63.5 0)
+    (property "LCSC" "C307331" (id 4) (at 167.64 63.5 0)
       (effects (font (size 1.27 1.27)) hide)
     )
@@
       (effects (font (size 1.27 1.27)) hide)
     )
-    (property "LCSC" "C1525" (id 4) (at 180.34 63.5 0)
+    (property "LCSC" "C307331" (id 4) (at 180.34 63.5 0)
       (effects (font (size 1.27 1.27)) hide)
     )
@@
       (effects (font (size 1.27 1.27)) hide)
     )
-    (property "LCSC" "C52923" (id 4) (at 218.44 63.5 0)
+    (property "LCSC" "C20539426" (id 4) (at 218.44 63.5 0)
       (effects (font (size 1.27 1.27)) hide)
     )
@@
       (effects (font (size 1.27 1.27)) hide)
     )
-    (property "LCSC" "C1525" (id 4) (at 231.14 63.5 0)
+    (property "LCSC" "C307331" (id 4) (at 231.14 63.5 0)
       (effects (font (size 1.27 1.27)) hide)
     )
@@
       (effects (font (size 1.27 1.27)) hide)
     )
-    (property "LCSC" "C1525" (id 4) (at 175.26 78.74 0)
+    (property "LCSC" "C307331" (id 4) (at 175.26 78.74 0)
       (effects (font (size 1.27 1.27)) hide)
     )
@@
       (effects (font (size 1.27 1.27)) hide)
     )
-    (property "LCSC" "C25744" (id 4) (at 246.38 177.8 0)
+    (property "LCSC" "C2906861" (id 4) (at 246.38 177.8 0)
       (effects (font (size 1.27 1.27)) hide)
     )
@@
       (effects (font (size 1.27 1.27)) hide)
     )
-    (property "LCSC" "C25744" (id 4) (at 167.64 157.48 0)
+    (property "LCSC" "C2906861" (id 4) (at 167.64 157.48 0)
       (effects (font (size 1.27 1.27)) hide)
     )
@@
       (effects (font (size 1.27 1.27)) hide)
     )
-    (property "LCSC" "C25744" (id 4) (at 167.64 160.02 0)
+    (property "LCSC" "C2906861" (id 4) (at 167.64 160.02 0)
       (effects (font (size 1.27 1.27)) hide)
     )
@@
       (effects (font (size 1.27 1.27)) hide)
     )
-    (property "LCSC" "C25744" (id 4) (at 167.64 162.56 0)
+    (property "LCSC" "C2906861" (id 4) (at 167.64 162.56 0)
       (effects (font (size 1.27 1.27)) hide)
     )
@@
       (effects (font (size 1.27 1.27)) hide)
     )
-    (property "LCSC" "C25744" (id 4) (at 238.76 106.68 0)
+    (property "LCSC" "C2906861" (id 4) (at 238.76 106.68 0)
       (effects (font (size 1.27 1.27)) hide)
     )
@@
       (effects (font (size 1.27 1.27)) hide)
     )
-    (property "LCSC" "C25744" (id 4) (at 238.76 109.22 0)
+    (property "LCSC" "C2906861" (id 4) (at 238.76 109.22 0)
       (effects (font (size 1.27 1.27)) hide)
     )
@@
       (effects (font (size 1.27 1.27)) hide)
     )
-    (property "LCSC" "C25744" (id 4) (at 238.76 111.76 0)
+    (property "LCSC" "C2906861" (id 4) (at 238.76 111.76 0)
       (effects (font (size 1.27 1.27)) hide)
     )
@@
       (effects (font (size 1.27 1.27)) hide)
     )
-    (property "LCSC" "C25744" (id 4) (at 238.76 119.38 0)
+    (property "LCSC" "C2906861" (id 4) (at 238.76 119.38 0)
       (effects (font (size 1.27 1.27)) hide)
     )
@@
       (effects (font (size 1.27 1.27)) hide)
     )
-    (property "LCSC" "C25744" (id 4) (at 238.76 149.86 0)
+    (property "LCSC" "C2906861" (id 4) (at 238.76 149.86 0)
       (effects (font (size 1.27 1.27)) hide)
     )
@@
       (effects (font (size 1.27 1.27)) hide)
     )
-    (property "LCSC" "C25744" (id 4) (at 238.76 170.18 0)
+    (property "LCSC" "C2906861" (id 4) (at 238.76 170.18 0)
       (effects (font (size 1.27 1.27)) hide)
     )
@@
       (effects (font (size 1.27 1.27)) hide)
     )
-    (property "LCSC" "C25744" (id 4) (at 167.64 139.7 0)
+    (property "LCSC" "C2906861" (id 4) (at 167.64 139.7 0)
       (effects (font (size 1.27 1.27)) hide)
     )
@@
       (effects (font (size 1.27 1.27)) hide)
     )
-    (property "LCSC" "C25744" (id 4) (at 167.64 142.24 0)
+    (property "LCSC" "C2906861" (id 4) (at 167.64 142.24 0)
       (effects (font (size 1.27 1.27)) hide)
     )
@@
       (effects (font (size 1.27 1.27)) hide)
     )
-    (property "LCSC" "C25744" (id 4) (at 238.76 127.0 0)
+    (property "LCSC" "C2906861" (id 4) (at 238.76 127.0 0)
       (effects (font (size 1.27 1.27)) hide)
     )
@@
       (effects (font (size 1.27 1.27)) hide)
     )
-    (property "LCSC" "C25744" (id 4) (at 167.64 154.94 0)
+    (property "LCSC" "C2906861" (id 4) (at 167.64 154.94 0)
       (effects (font (size 1.27 1.27)) hide)
     )
@@
       (effects (font (size 1.27 1.27)) hide)
     )
-    (property "LCSC" "C25744" (id 4) (at 167.64 119.38 0)
+    (property "LCSC" "C2906861" (id 4) (at 167.64 119.38 0)
       (effects (font (size 1.27 1.27)) hide)
     )
@@
       (effects (font (size 1.27 1.27)) hide)
     )
-    (property "LCSC" "C25744" (id 4) (at 238.76 154.94 0)
+    (property "LCSC" "C2906861" (id 4) (at 238.76 154.94 0)
       (effects (font (size 1.27 1.27)) hide)
     )
@@
       (effects (font (size 1.27 1.27)) hide)
     )
-    (property "LCSC" "C25744" (id 4) (at 238.76 157.48 0)
-      (effects (font (size 1.27 1.27)) hide)
-    )
+    (property "LCSC" "C2906861" (id 4) (at 238.76 157.48 0)
+      (effects (font (size 1.27 1.27)) hide)
+    )
