File: 01_hardware/kicad_project/pri_aux.kicad_sch (KiCad schematic)
At the start: 20 parts, among them U12 CA-IS3642LVW, U13 LMR16006XDDCR, U14 AMS1117-5.0

Commit message: update D
Parts:
- added C79: 1n C0G, Capacitor_SMD:C_0402_1005Metric, symbol Device:C
- added C80: 100n, Capacitor_SMD:C_0402_1005Metric, symbol Device:C
- added R81: 191k 1%, Resistor_SMD:R_1206_3216Metric, symbol Device:R
- added R82: 10k 1%, Resistor_SMD:R_0402_1005Metric, symbol Device:R
- added R83: 10k, Resistor_SMD:R_0402_1005Metric, symbol Device:R
- added R84: 2.2M, Resistor_SMD:R_0402_1005Metric, symbol Device:R
- added R85: 1k, Resistor_SMD:R_0402_1005Metric, symbol Device:R
- added TP1: VIN, TestPoint:TestPoint_Pad_D1.5mm, symbol Connector:TestPoint
- added TP2: GNDP, TestPoint:TestPoint_Pad_D1.5mm, symbol Connector:TestPoint
- added TP3: +10V_P, TestPoint:TestPoint_Pad_D1.5mm, symbol Connector:TestPoint
- added TP4: +5V_P, TestPoint:TestPoint_Pad_D1.5mm, symbol Connector:TestPoint
- added U15: LMV331IDBVR, Package_TO_SOT_SMD:SOT-23-5, symbol Comparator:LMV331
- added U16: TL431AIDBZR, Package_TO_SOT_SMD:SOT-23, symbol Reference_Voltage:TL431DBZ
- D6: value B1100 -> SS110; footprint Diode_SMD:D_SOD-123F -> Diode_SMD:D_SMA; LCSC (none) -> C224219; MPN B1100 / SS110 -> SS110
Connections:
- net +10V_P: now also TP3.1
- net +5V_P: now also C80.1, R83.1, R85.1, TP4.1, U15.5 (V+)
- net GNDP: now also C79.2, C80.2, R82.2, TP2.1, U15.2 (V-), U16.3 (A); no longer U12.3 (VI1)
- net VIN: now also R81.1, TP1.1
- net VIN_OVP: now reaches U12.14 (VO1)
- new net OVP_DIV: C79.1, R81.2, R82.1, R84.2, U15.1 (+)
- new net OVP_P: R83.2, R84.1, U12.3 (VI1), U15.4
- new net VREF_P: R85.2, U15.3 (-), U16.1 (K), U16.2 (REF)
- no-connect marks 2 -> 1
Other:
- note added: "INPUT OVP (primary side) Trip = 2.495 V x (1 + 191k/10k) = 50.2 V rising Hysteresis ~0.4 V (R84 2.2M) OVP_P high = over-voltage -> U12 VI1 -> VO1 -> VIN_OVP -> PA15 (HRTIM1_FLT2 / EXTI15)"
