File: 01_hardware/kicad_project/pri_aux.kicad_sch (KiCad schematic)
At the start: 33 parts, among them U12 CA-IS3642LVW, U13 LMR16006XDDCR, U14 AMS1117-5.0, U15 LMV331IDBVR, U16 TL431AIDBZR

Commit message: VIN monitor: sawtooth/comparator PWM over spare isolator channel to PA2 (TIM15_CH1)
- Primary: PNP current-source ramp (~5 ms) into 47 nF C0G, U17 reset detector,
  U18 PWM comparator vs OVP_DIV; R81/R82 now 0.1 %
- U12 VI2->VO2 carries VIN_PWM to PA2; R93 is its pull-down
- PCB: new block placed/routed below U15/U16, R106 moved for courtyard,
  GNDP island vias, silkscreen for new parts; DRC clean, netlist parity OK
- Outputs regenerated (BOM, Gerbers, CPL, EasyEDA, PDFs, pin-map)

Co-Authored-By: Claude Opus 5.5 <noreply@anthropic.com>
Claude-Session: https://claude.ai/code/session_01A35wrnwFKLPSaRSxxHs471
Parts:
- added C81: 1n, Capacitor_SMD:C_0402_1005Metric, symbol Device:C
- added C82: 47n C0G 50V, Capacitor_SMD:C_0805_2012Metric, symbol Device:C
- added C83, C84: 100n, Capacitor_SMD:C_0402_1005Metric, symbol Device:C
- added D7: 1N4148W, Diode_SMD:D_SOD-123, symbol Device:D
- added Q10: 2N7002, Package_TO_SOT_SMD:SOT-23, symbol Transistor_FET:2N7002
- added Q9: MMBT3906, Package_TO_SOT_SMD:SOT-23, symbol Transistor_BJT:MMBT3906
- added R106: 1k, Resistor_SMD:R_0402_1005Metric, symbol Device:R
- added R107: 22k, Resistor_SMD:R_0402_1005Metric, symbol Device:R
- added R108, R109: 10k, Resistor_SMD:R_0402_1005Metric, symbol Device:R
- added R110: 1M, Resistor_SMD:R_0402_1005Metric, symbol Device:R
- added R86: 56k 1%, Resistor_SMD:R_0402_1005Metric, symbol Device:R
- added R87: 10k 1%, Resistor_SMD:R_0402_1005Metric, symbol Device:R
- added R88: 15k 1%, Resistor_SMD:R_0402_1005Metric, symbol Device:R
- added R89: 22R, Resistor_SMD:R_0402_1005Metric, symbol Device:R
- added U17, U18: LMV331IDBVR, Package_TO_SOT_SMD:SOT-23-5, symbol Comparator:LMV331
- R81: value 191k 1% -> 191k 0.1%; MPN 191k 1% -> 191k 0.1%
- R82: value 10k 1% -> 10k 0.1%; MPN 10k 1% -> 10k 0.1%
Connections:
- net +5V_P: now also C83.1, C84.1, R106.1, R108.1, R86.1, R87.1, U17.5 (V+), U18.5 (V+)
- net GNDP: now also C81.2, C82.2, C83.2, C84.2, Q10.2 (S), R107.2, R88.2, U17.2 (V-), U18.2 (V-); no longer U12.4 (VI2)
- net OVP_DIV: now also U18.3 (-)
- net VREF_P: now also U17.3 (-)
- net VIN_PWM: now reaches U12.13 (VO2)
- new net DIS_P: Q10.3 (D), R89.1
- new net GATE_P: C81.1, D7.1 (K), Q10.1 (G), R107.1
- new net PB_P: Q9.1 (B), R87.2, R88.1
- new net PE_P: Q9.2 (E), R86.2
- new net RAMPS_P: R109.2, R110.2, U18.1 (+)
- new net RAMP_P: C82.1, Q9.3 (C), R109.1, R89.2, U17.1 (+)
- new net RST_P: D7.2 (A), R106.2, U17.4
- new net VINPWM_P: R108.2, R110.1, U12.4 (VI2), U18.4
- no-connect marks 1 -> 0
Other:
- note added: "VIN MONITOR (primary side, monitoring only) Ramp 0 -> 2.495 V in ~5 ms (Q9 ~24 uA into C82 47n C0G), reset ~20 us by U17/D7/C81/Q10 U18: VINPWM_P high while RAMP > OVP_DIV -> U12 VI2 -> VO2 -> VIN_PWM -> PA2 (TIM15_CH1 PWM input) VIN = 50.36 V x (T_ramp - t_high) / T_ramp, T_ramp = period - t_reset; calibrate once"

Commit message: Review fixes: VIN monitor linearity and reset, full-scale summary, design notes
- U18 inputs swapped (IN+ = OVP_DIV, IN- = RAMP via R109 1k); R110 4.7M
  hysteresis now on the divider, not the ramp (old 1M path bent the ramp:
  +12.5 % error at 12 V; now < 0.02 % in simulation)
- Reset pulse hardened: C81 220p C0G, R107 100k so C82 always fully discharges
- OVP trip corrected to 50.26 V rising / 49.83 V falling; TL431A noted as 1 %
- PCB re-routed locally, values synced to schematic; DRC clean, parity OK,
  isolation 4.0 mm
- Design notes: full-scale and threshold summary, VIN monitor firmware formula
  and two-point calibration; exported to DOCX and PDF
- Pin-map, BOM, Gerbers, CPL, EasyEDA zip and PDFs regenerated

Co-Authored-By: Claude Opus 5.5 <noreply@anthropic.com>
Claude-Session: https://claude.ai/code/session_01A35wrnwFKLPSaRSxxHs471
Parts:
- C81: value 1n -> 220p C0G; MPN 1n -> 220p C0G
- R107: value 22k -> 100k; MPN 22k -> 100k
- R109: value 10k -> 1k; MPN 10k -> 1k
- R110: value 1M -> 4.7M; MPN 1M -> 4.7M
Connections:
- net OVP_DIV: now also R110.2, U18.1 (+); no longer U18.3 (-)
- net RAMPS_P: now also U18.3 (-); no longer R110.2, U18.1 (+)
Other:
- note added: "VIN MONITOR (primary side, monitoring only) Ramp 0 -> 2.495 V in ~5 ms (Q9 ~24 uA into C82 47n C0G), reset ~20 us by U17/D7/C81/Q10 U18: VINPWM_P high while RAMP < OVP_DIV (R110 hysteresis on the divider side) -> U12 VI2 -> VO2 -> VIN_PWM -> PA2 (TIM15_CH1 PWM input) VIN = 50.47 V x (t_high - t_reset) / (period - t_reset) - 0.20 V, t_reset ~20 us; calibrate once"
- note removed: "VIN MONITOR (primary side, monitoring only) Ramp 0 -> 2.495 V in ~5 ms (Q9 ~24 uA into C82 47n C0G), reset ~20 us by U17/D7/C81/Q10 U18: VINPWM_P high while RAMP > OVP_DIV -> U12 VI2 -> VO2 -> VIN_PWM -> PA2 (TIM15_CH1 PWM input) VIN = 50.36 V x (T_ramp - t_high) / T_ramp, T_ramp = period - t_reset; calibrate once"
Changed lines of the file:
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@@
   (junction (at 236.22 158.75) (diameter 0) (color 0 0 0 0)
   )
-  (junction (at 236.22 218.44) (diameter 0) (color 0 0 0 0)
-  )
-  (junction (at 256.54 215.9) (diameter 0) (color 0 0 0 0)
+  (junction (at 256.54 214.63) (diameter 0) (color 0 0 0 0)
   )
   (wire (pts (xy 88.9 78.74) (xy 91.44 78.74))
@@
     (stroke (width 0) (type default))
   )
-  (wire (pts (xy 219.71 218.44) (xy 217.17 218.44))
-    (stroke (width 0) (type default))
-  )
-  (wire (pts (xy 227.33 218.44) (xy 229.87 218.44))
+  (wire (pts (xy 219.71 223.52) (xy 217.17 223.52))
+    (stroke (width 0) (type default))
+  )
+  (wire (pts (xy 227.33 223.52) (xy 229.87 223.52))
     (stroke (width 0) (type default))
   )
@@
     (stroke (width 0) (type default))
   )
+  (wire (pts (xy 229.87 223.52) (xy 236.22 223.52))
+    (stroke (width 0) (type default))
+  )
   (wire (pts (xy 137.16 100.33) (xy 116.84 100.33))
     (stroke (width 0) (type default))
@@
     (stroke (width 0) (type default))
   )
-  (wire (pts (xy 229.87 218.44) (xy 236.22 218.44))
-    (stroke (width 0) (type default))
-  )
-  (wire (pts (xy 252.73 205.74) (xy 252.73 214.63))
-    (stroke (width 0) (type default))
-  )
-  (wire (pts (xy 252.73 214.63) (xy 236.22 214.63))
-    (stroke (width 0) (type default))
-  )
-  (wire (pts (xy 236.22 214.63) (xy 236.22 218.44))
-    (stroke (width 0) (type default))
-  )
   (wire (pts (xy 266.7 214.63) (xy 256.54 214.63))
     (stroke (width 0) (type default))
   )
-  (wire (pts (xy 256.54 214.63) (xy 256.54 215.9))
-    (stroke (width 0) (type default))
-  )
-  (wire (pts (xy 256.54 215.9) (xy 256.54 220.98))
-    (stroke (width 0) (type default))
-  )
-  (wire (pts (xy 240.03 205.74) (xy 240.03 215.9))
-    (stroke (width 0) (type default))
-  )
-  (wire (pts (xy 240.03 215.9) (xy 256.54 215.9))
+  (wire (pts (xy 256.54 214.63) (xy 256.54 220.98))
+    (stroke (width 0) (type default))
+  )
+  (wire (pts (xy 240.03 205.74) (xy 240.03 214.63))
+    (stroke (width 0) (type default))
+  )
+  (wire (pts (xy 240.03 214.63) (xy 256.54 214.63))
     (stroke (width 0) (type default))
   )
@@
     (effects (font (size 1.27 1.27)) (justify left top))
   )
-  (text "VIN MONITOR (primary side, monitoring only)\nRamp 0 -> 2.495 V in ~5 ms (Q9 ~24 uA into C82 47n C0G), reset ~20 us by U17/D7/C81/Q10\nU18: VINPWM_P high while RAMP > OVP_DIV  ->  U12 VI2 -> VO2 -> VIN_PWM -> PA2 (TIM15_CH1 PWM input)\nVIN = 50.36 V x (T_ramp - t_high) / T_ramp,  T_ramp = period - t_reset; calibrate once"
+  (text "VIN MONITOR (primary side, monitoring only)\nRamp 0 -> 2.495 V in ~5 ms (Q9 ~24 uA into C82 47n C0G), reset ~20 us by U17/D7/C81/Q10\nU18: VINPWM_P high while RAMP < OVP_DIV (R110 hysteresis on the divider side)  ->  U12 VI2 -> VO2 -> VIN_PWM -> PA2 (TIM15_CH1 PWM input)\nVIN = 50.47 V x (t_high - t_reset) / (period - t_reset) - 0.20 V,  t_reset ~20 us; calibrate once"
     (at 40.64 256.54 0)
     (effects (font (size 1.27 1.27)) (justify left top))
@@
     (effects (font (size 1.0 1.0)) (justify left bottom))
   )
+  (label "RAMPS_P" (at 229.87 223.52 0)
+    (effects (font (size 1.0 1.0)) (justify left bottom))
+  )
   (label "FB_P" (at 91.44 88.9 0)
     (effects (font (size 1.0 1.0)) (justify left bottom))
@@
     (effects (font (size 1.0 1.0)) (justify left bottom))
   )
-  (label "RAMPS_P" (at 252.73 205.74 0)
-    (effects (font (size 1.0 1.0)) (justify left bottom))
-  )
   (label "VINPWM_P" (at 240.03 205.74 180)
     (effects (font (size 1.0 1.0)) (justify right bottom))
@@
     (effects (font (size 1.0 1.0)) (justify right bottom))
   )
-  (label "RAMP_P" (at 217.17 218.44 180)
+  (label "RAMP_P" (at 217.17 223.52 180)
     (effects (font (size 1.0 1.0)) (justify right bottom))
   )
-  (label "OVP_DIV" (at 236.22 223.52 180)
+  (label "OVP_DIV" (at 236.22 218.44 180)
     (effects (font (size 1.0 1.0)) (justify right bottom))
+  )
+  (label "OVP_DIV" (at 252.73 205.74 0)
+    (effects (font (size 1.0 1.0)) (justify left bottom))
   )
   (label "GATE_P" (at 190.5 229.87 90)
@@
   (symbol (lib_id "Device:C") (at 190.5 236.22 0) (unit 1)
     (in_bom yes) (on_board yes)
-    (property "Reference" "C81" (id 0) (at 195.035 235.204 0)
-      (effects (font (size 1.27 1.27)))
-    )
-    (property "Value" "1n" (id 1) (at 194.202 237.02 0)
+    (property "Reference" "C81" (id 0) (at 185.965 235.204 0)
+      (effects (font (size 1.27 1.27)))
+    )
+    (property "Value" "220p C0G" (id 1) (at 184.038 237.02 0)
       (effects (font (size 1.0 1.0)))
     )
@@
       (effects (font (size 1.27 1.27)) hide)
     )
-    (property "MPN" "1n" (id 5) (at 190.5 236.22 0)
+    (property "MPN" "220p C0G" (id 5) (at 190.5 236.22 0)
       (effects (font (size 1.27 1.27)) hide)
     )
@@
       (effects (font (size 1.27 1.27)))
     )
-    (property "Value" "22k" (id 1) (at 203.806 237.02 0)
+    (property "Value" "100k" (id 1) (at 204.266 237.02 0)
       (effects (font (size 1.0 1.0)))
     )
@@
       (effects (font (size 1.27 1.27)) hide)
     )
-    (property "MPN" "22k" (id 5) (at 200.66 236.22 0)
+    (property "MPN" "100k" (id 5) (at 200.66 236.22 0)
       (effects (font (size 1.27 1.27)) hide)
     )
@@
     (pin "2")
   )
-  (symbol (lib_id "Device:R") (at 223.52 218.44 90) (unit 1)
-    (in_bom yes) (on_board yes)
-    (property "Reference" "R109" (id 0) (at 223.52 215.808 90)
-      (effects (font (size 1.27 1.27)))
-    )
-    (property "Value" "10k" (id 1) (at 223.52 220.856 90)
-      (effects (font (size 1.0 1.0)))
-    )
-    (property "Footprint" "Resistor_SMD:R_0402_1005Metric" (id 2) (at 223.52 218.44 0)
-      (effects (font (size 1.27 1.27)) hide)
-    )
-    (property "Datasheet" "" (id 3) (at 223.52 218.44 0)
-      (effects (font (size 1.27 1.27)) hide)
-    )
-    (property "LCSC" "" (id 4) (at 223.52 218.44 0)
-      (effects (font (size 1.27 1.27)) hide)
-    )
-    (property "MPN" "10k" (id 5) (at 223.52 218.44 0)
+  (symbol (lib_id "Device:R") (at 223.52 223.52 90) (unit 1)
+    (in_bom yes) (on_board yes)
+    (property "Reference" "R109" (id 0) (at 223.52 220.888 90)
+      (effects (font (size 1.27 1.27)))
+    )
+    (property "Value" "1k" (id 1) (at 223.52 225.936 90)
+      (effects (font (size 1.0 1.0)))
+    )
+    (property "Footprint" "Resistor_SMD:R_0402_1005Metric" (id 2) (at 223.52 223.52 0)
+      (effects (font (size 1.27 1.27)) hide)
+    )
+    (property "Datasheet" "" (id 3) (at 223.52 223.52 0)
+      (effects (font (size 1.27 1.27)) hide)
+    )
+    (property "LCSC" "" (id 4) (at 223.52 223.52 0)
+      (effects (font (size 1.27 1.27)) hide)
+    )
+    (property "MPN" "1k" (id 5) (at 223.52 223.52 0)
       (effects (font (size 1.27 1.27)) hide)
     )
@@
       (effects (font (size 1.27 1.27)))
     )
-    (property "Value" "1M" (id 1) (at 246.38 203.324 90)
+    (property "Value" "4.7M" (id 1) (at 246.38 203.324 90)
       (effects (font (size 1.0 1.0)))
     )
@@
       (effects (font (size 1.27 1.27)) hide)
     )
-    (property "MPN" "1M" (id 5) (at 246.38 205.74 0)
-      (effects (font (size 1.27 1.27)) hide)
-    )
+    (property "MPN" "4.7M" (id 5) (at 246.38 205.74 0)
+      (effects (font (size 1.27 1.27)) hide)
+    )
