File: 01_hardware/kicad_project/sbb.kicad_sch (KiCad schematic)
At the start: 45 parts, among them J2 VOUT 1.5-48V, Q1 NCEP0140AG, Q2 NCEP0160AG, Q3 NCEP0160AG, Q4 NCEP0140AG, U2 UCC27211DDAR, U3 UCC27211DDAR

Commit message: update D
Parts:
- added TP11: VOUT, TestPoint:TestPoint_Pad_D1.5mm, symbol Connector:TestPoint
- added TP12: GND, TestPoint:TestPoint_Pad_D1.5mm, symbol Connector:TestPoint
Connections:
- net GND: now also TP12.1
- net VOUT: now also TP11.1
