File: 01_hardware/kicad_project/sbb.kicad_sch (KiCad schematic)
At the start: 47 parts, among them J2 VOUT 1.5-48V, Q1 NCEP0140AG, Q2 NCEP0160AG, Q3 NCEP0160AG, Q4 NCEP0140AG, U2 UCC27211DDAR, U3 UCC27211DDAR

Commit message: Rev D order prep: common F1/L2/L3 parts, JLC-checked LCSC numbers, assembly files
- F1: 2512 -> 1206 7 A 63 V fuse (Littelfuse 0458007.DR, C206980; 2nd source Schurter 3413.0326.11)
- L2/L3: SRP5030 -> 5040 shielded 47 uH (SWPA5040S470MT, C86617; 2nd source SRN5040-470M, NRS5040T470MMGK)
- EN_AUX re-routed off the L2 pad gap; VIN track centred between the L3 pads (0.4 mm each side)
- LCSC numbers checked in the JLCPCB library for every assembled part (design.py JLC_LCSC),
  written to the BOMs, schematic and PCB fields
- New JLC assembly upload files DCDC_JLC_BOM.csv / DCDC_JLC_CPL.csv (217 parts; U1, T1,
  connectors, headers and SW1 hand-soldered) and jlc_order_files.py to rebuild them
- 03_calculations/aux_fuse_check.py: aux inductor peak 0.27 A vs 1.1 A Isat; F1 4.8 A at 12 V / 50 W
- Design notes (docx/pdf), README, Gerbers, CPL, PDFs and DRC report regenerated
- Checks: DRC (JLC rules) 0 errors / 0 unconnected, netlist 134 nets / 257 parts 0 errors,
  isolation check 0 errors, silkscreen clean

Co-Authored-By: Claude Opus 5.5 <noreply@anthropic.com>
Claude-Session: https://claude.ai/code/session_01A35wrnwFKLPSaRSxxHs471
Parts:
- C1, C11: LCSC (none) -> C249664
- C10, C2, C3, C4, C5, C7, C8, C9: LCSC (none) -> C153036
- C12, C6: LCSC (none) -> C88219
- C15: LCSC (none) -> C14663
- C16, C18: LCSC (none) -> C15849
- C17, C19: LCSC (none) -> C307331
- C20, R10, R4: LCSC (none) -> C23164
- R1: LCSC (none) -> C2907507
- R11, R12, R13, R14, R5, R6, R7, R8: LCSC (none) -> C25744
- R9: LCSC (none) -> C141980
- RS1: LCSC (none) -> C500738
- RSH1: LCSC (none) -> C500718
- U3: LCSC C141980 -> C14663
Changed lines of the file:
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@@
       (effects (font (size 1.27 1.27)) hide)
     )
-    (property "LCSC" "" (id 4) (at 25.4 45.72 0)
+    (property "LCSC" "C249664" (id 4) (at 25.4 45.72 0)
       (effects (font (size 1.27 1.27)) hide)
     )
@@
       (effects (font (size 1.27 1.27)) hide)
     )
-    (property "LCSC" "" (id 4) (at 43.18 45.72 0)
+    (property "LCSC" "C153036" (id 4) (at 43.18 45.72 0)
       (effects (font (size 1.27 1.27)) hide)
     )
@@
       (effects (font (size 1.27 1.27)) hide)
     )
-    (property "LCSC" "" (id 4) (at 60.96 45.72 0)
+    (property "LCSC" "C153036" (id 4) (at 60.96 45.72 0)
       (effects (font (size 1.27 1.27)) hide)
     )
@@
       (effects (font (size 1.27 1.27)) hide)
     )
-    (property "LCSC" "" (id 4) (at 78.74 45.72 0)
+    (property "LCSC" "C153036" (id 4) (at 78.74 45.72 0)
       (effects (font (size 1.27 1.27)) hide)
     )
@@
       (effects (font (size 1.27 1.27)) hide)
     )
-    (property "LCSC" "" (id 4) (at 96.52 45.72 0)
+    (property "LCSC" "C153036" (id 4) (at 96.52 45.72 0)
       (effects (font (size 1.27 1.27)) hide)
     )
@@
       (effects (font (size 1.27 1.27)) hide)
     )
-    (property "LCSC" "" (id 4) (at 114.3 45.72 0)
+    (property "LCSC" "C88219" (id 4) (at 114.3 45.72 0)
       (effects (font (size 1.27 1.27)) hide)
     )
@@
       (effects (font (size 1.27 1.27)) hide)
     )
-    (property "LCSC" "" (id 4) (at 152.4 139.7 0)
+    (property "LCSC" "C500738" (id 4) (at 152.4 139.7 0)
       (effects (font (size 1.27 1.27)) hide)
     )
@@
       (effects (font (size 1.27 1.27)) hide)
     )
-    (property "LCSC" "" (id 4) (at 190.5 167.64 0)
+    (property "LCSC" "C153036" (id 4) (at 190.5 167.64 0)
       (effects (font (size 1.27 1.27)) hide)
     )
@@
       (effects (font (size 1.27 1.27)) hide)
     )
-    (property "LCSC" "" (id 4) (at 208.28 167.64 0)
+    (property "LCSC" "C153036" (id 4) (at 208.28 167.64 0)
       (effects (font (size 1.27 1.27)) hide)
     )
@@
       (effects (font (size 1.27 1.27)) hide)
     )
-    (property "LCSC" "" (id 4) (at 226.06 167.64 0)
+    (property "LCSC" "C153036" (id 4) (at 226.06 167.64 0)
       (effects (font (size 1.27 1.27)) hide)
     )
@@
       (effects (font (size 1.27 1.27)) hide)
     )
-    (property "LCSC" "" (id 4) (at 243.84 167.64 0)
+    (property "LCSC" "C153036" (id 4) (at 243.84 167.64 0)
       (effects (font (size 1.27 1.27)) hide)
     )
@@
       (effects (font (size 1.27 1.27)) hide)
     )
-    (property "LCSC" "" (id 4) (at 261.62 167.64 0)
+    (property "LCSC" "C249664" (id 4) (at 261.62 167.64 0)
       (effects (font (size 1.27 1.27)) hide)
     )
@@
       (effects (font (size 1.27 1.27)) hide)
     )
-    (property "LCSC" "" (id 4) (at 279.4 167.64 0)
+    (property "LCSC" "C88219" (id 4) (at 279.4 167.64 0)
       (effects (font (size 1.27 1.27)) hide)
     )
@@
       (effects (font (size 1.27 1.27)) hide)
     )
-    (property "LCSC" "" (id 4) (at 307.34 180.34 0)
+    (property "LCSC" "C500718" (id 4) (at 307.34 180.34 0)
       (effects (font (size 1.27 1.27)) hide)
     )
@@
       (effects (font (size 1.27 1.27)) hide)
     )
-    (property "LCSC" "" (id 4) (at 297.18 167.64 0)
+    (property "LCSC" "C2907507" (id 4) (at 297.18 167.64 0)
       (effects (font (size 1.27 1.27)) hide)
     )
@@
       (effects (font (size 1.27 1.27)) hide)
     )
-    (property "LCSC" "" (id 4) (at 76.2 81.28 0)
+    (property "LCSC" "C14663" (id 4) (at 76.2 81.28 0)
       (effects (font (size 1.27 1.27)) hide)
     )
@@
       (effects (font (size 1.27 1.27)) hide)
     )
-    (property "LCSC" "" (id 4) (at 30.48 86.36 0)
+    (property "LCSC" "C15849" (id 4) (at 30.48 86.36 0)
       (effects (font (size 1.27 1.27)) hide)
     )
@@
       (effects (font (size 1.27 1.27)) hide)
     )
-    (property "LCSC" "" (id 4) (at 38.1 86.36 0)
+    (property "LCSC" "C307331" (id 4) (at 38.1 86.36 0)
       (effects (font (size 1.27 1.27)) hide)
     )
@@
       (effects (font (size 1.27 1.27)) hide)
     )
-    (property "LCSC" "" (id 4) (at 93.98 76.2 0)
+    (property "LCSC" "C23164" (id 4) (at 93.98 76.2 0)
       (effects (font (size 1.27 1.27)) hide)
     )
@@
       (effects (font (size 1.27 1.27)) hide)
     )
-    (property "LCSC" "" (id 4) (at 93.98 114.3 0)
+    (property "LCSC" "C25744" (id 4) (at 93.98 114.3 0)
       (effects (font (size 1.27 1.27)) hide)
     )
@@
       (effects (font (size 1.27 1.27)) hide)
     )
-    (property "LCSC" "" (id 4) (at 104.14 86.36 0)
+    (property "LCSC" "C25744" (id 4) (at 104.14 86.36 0)
       (effects (font (size 1.27 1.27)) hide)
     )
@@
       (effects (font (size 1.27 1.27)) hide)
     )
-    (property "LCSC" "" (id 4) (at 104.14 124.46 0)
+    (property "LCSC" "C25744" (id 4) (at 104.14 124.46 0)
       (effects (font (size 1.27 1.27)) hide)
     )
@@
       (effects (font (size 1.27 1.27)) hide)
     )
-    (property "LCSC" "" (id 4) (at 30.48 116.84 0)
+    (property "LCSC" "C25744" (id 4) (at 30.48 116.84 0)
       (effects (font (size 1.27 1.27)) hide)
     )
@@
       (effects (font (size 1.27 1.27)) hide)
     )
-    (property "LCSC" "" (id 4) (at 38.1 116.84 0)
+    (property "LCSC" "C141980" (id 4) (at 38.1 116.84 0)
       (effects (font (size 1.27 1.27)) hide)
     )
@@
       (effects (font (size 1.27 1.27)) hide)
     )
-    (property "LCSC" "C141980" (id 4) (at 248.92 96.52 0)
+    (property "LCSC" "C14663" (id 4) (at 248.92 96.52 0)
       (effects (font (size 1.27 1.27)) hide)
     )
@@
       (effects (font (size 1.27 1.27)) hide)
     )
-    (property "LCSC" "" (id 4) (at 231.14 81.28 0)
+    (property "LCSC" "C15849" (id 4) (at 231.14 81.28 0)
       (effects (font (size 1.27 1.27)) hide)
     )
@@
       (effects (font (size 1.27 1.27)) hide)
     )
-    (property "LCSC" "" (id 4) (at 276.86 86.36 0)
+    (property "LCSC" "C307331" (id 4) (at 276.86 86.36 0)
       (effects (font (size 1.27 1.27)) hide)
     )
@@
       (effects (font (size 1.27 1.27)) hide)
     )
-    (property "LCSC" "" (id 4) (at 284.48 86.36 0)
+    (property "LCSC" "C23164" (id 4) (at 284.48 86.36 0)
       (effects (font (size 1.27 1.27)) hide)
     )
@@
       (effects (font (size 1.27 1.27)) hide)
     )
-    (property "LCSC" "" (id 4) (at 210.82 76.2 0)
+    (property "LCSC" "C23164" (id 4) (at 210.82 76.2 0)
       (effects (font (size 1.27 1.27)) hide)
     )
@@
       (effects (font (size 1.27 1.27)) hide)
     )
-    (property "LCSC" "" (id 4) (at 210.82 114.3 0)
+    (property "LCSC" "C25744" (id 4) (at 210.82 114.3 0)
       (effects (font (size 1.27 1.27)) hide)
     )
@@
       (effects (font (size 1.27 1.27)) hide)
     )
-    (property "LCSC" "" (id 4) (at 200.66 86.36 0)
+    (property "LCSC" "C25744" (id 4) (at 200.66 86.36 0)
       (effects (font (size 1.27 1.27)) hide)
     )
@@
       (effects (font (size 1.27 1.27)) hide)
     )
-    (property "LCSC" "" (id 4) (at 200.66 124.46 0)
+    (property "LCSC" "C25744" (id 4) (at 200.66 124.46 0)
       (effects (font (size 1.27 1.27)) hide)
     )
@@
       (effects (font (size 1.27 1.27)) hide)
     )
-    (property "LCSC" "" (id 4) (at 276.86 116.84 0)
-      (effects (font (size 1.27 1.27)) hide)
-    )
+    (property "LCSC" "C25744" (id 4) (at 276.86 116.84 0)
+      (effects (font (size 1.27 1.27)) hide)
+    )

Commit message: Rev E: isolated flyback aux supply, VREF+ back to 3.3 V, 1 oz re-layout
- New isolated aux flyback (sheet iso_pwr): UC3843B U20 from +10V_P, FDN86246 Q11,
  PA3855.006NLT EP13 T2, SS110 D9 -> isolated +10 V; secondary regulation TL431 U22 +
  EL357N opto U21 into COMP; RCD clamp D8/R116/C94; 2 A primary limit (R114)
- Secondary rails from the flyback, not VBUS: +10 V -> U4 10->5 V -> U5 TLV75533 3.3 V;
  MCU, CAN and drivers up before the LLC starts
- U12 -> CA-IS3742LW (data only); REF3030 U19 removed, VREF+ = +3V3A (3.3 V full scale)
- PCB re-placed / re-routed for 1 oz outer / 0.5 oz inner: power pours on F.Cu, In1 solid
  ground planes, gate loops as tight HO/HS pairs, 1.7 mm power-via pitch, per-pad GND vias
  in the MCU area; copper loss ~0.5 W at 50 W (03_calculations/copper_check.txt)
- DRC (JLC rules) 0 errors / 0 unconnected; netlist 148 nets / 284 parts 0 errors;
  isolation bands clear; BOM / JLC BOM+CPL / Gerbers / PDFs / design notes / READMEs updated
- Scripts: 04_scripts/pcb5 (placement, pours, routing, floods, island vias, silk),
  03_calculations/flyback_aux.py, copper_check.py

Co-Authored-By: Claude Opus 5.5 <noreply@anthropic.com>
Claude-Session: https://claude.ai/code/session_01A35wrnwFKLPSaRSxxHs471
Parts:
- added TP5: VBUS, TestPoint:TestPoint_Pad_D1.5mm, symbol Connector:TestPoint
- C18: LCSC C15849 -> C14663
- C19: LCSC C307331 -> C15849
- C20: LCSC C23164 -> C307331
- R11, R5: LCSC C25744 -> C23164
- R15: LCSC (none) -> C25744
- R9: LCSC C141980 -> C25744
- U3: LCSC C14663 -> C141980
Connections:
- net VBUS: now also TP5.1

Commit message: Rev E BOM: in-stock LCSC first source for every part; 2nd/3rd sources checked
- First sources swapped (same footprints, layout unchanged): U1 STM32G474RBT3,
  Q2/Q3/Q5/Q6 NCEP068N10G, 10k 0402 FOJAN, 100n 0402 merged onto C307331,
  1u 0402 CCTC, R62/R63/R89/R82, FB1 Murata BLM18KG601SN1D, L2/L3 cjiang
  FNR5040S470MT, C82 KEMET C0G (was X7R), RS1 Milliohm HoJLR2512, SS110 MDD
- LCSC part numbers for the hand-soldered headers (J1-J5, J7, JP1)
- Schematic and PCB fields, BOM, JLC BOM/CPL, PDFs and design notes regenerated;
  netlist check 0 errors, DRC unchanged
- BOM_sourcing_revE.xlsx: live LCSC stock 2026-10-20, 2nd/3rd sources checked
  for pinout / land pattern / ratings, PCB reserve options for T2 and U9

Co-Authored-By: Claude Opus 5.5 <noreply@anthropic.com>
Claude-Session: https://claude.ai/code/session_01A35wrnwFKLPSaRSxxHs471
Parts:
- J2: LCSC (none) -> C441204
- Q2, Q3: value NCEP0160AG -> NCEP068N10G; LCSC C503012 -> C503061; MPN NCEP0160AG -> NCEP068N10G
- R12, R13, R14, R15, R6, R7, R8, R9: LCSC C25744 -> C2906861
- RS1: LCSC C500738 -> C2904236; MPN 4m 1% 2W -> HoJLR2512-3W-4mR-1%
Changed lines of the file:
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@@
       (effects (font (size 1.27 1.27)))
     )
-    (property "Value" "NCEP0160AG" (id 1) (at 112.712 118.71 0)
+    (property "Value" "NCEP068N10G" (id 1) (at 112.712 118.71 0)
       (effects (font (size 1.27 1.27)))
     )
@@
       (effects (font (size 1.27 1.27)) hide)
     )
-    (property "LCSC" "C503012" (id 4) (at 116.84 114.3 0)
-      (effects (font (size 1.27 1.27)) hide)
-    )
-    (property "MPN" "NCEP0160AG" (id 5) (at 116.84 114.3 0)
+    (property "LCSC" "C503061" (id 4) (at 116.84 114.3 0)
+      (effects (font (size 1.27 1.27)) hide)
+    )
+    (property "MPN" "NCEP068N10G" (id 5) (at 116.84 114.3 0)
       (effects (font (size 1.27 1.27)) hide)
     )
@@
       (effects (font (size 1.27 1.27)))
     )
-    (property "Value" "NCEP0160AG" (id 1) (at 192.088 71.79 0)
+    (property "Value" "NCEP068N10G" (id 1) (at 192.088 71.79 0)
       (effects (font (size 1.27 1.27)))
     )
@@
       (effects (font (size 1.27 1.27)) hide)
     )
-    (property "LCSC" "C503012" (id 4) (at 187.96 76.2 0)
-      (effects (font (size 1.27 1.27)) hide)
-    )
-    (property "MPN" "NCEP0160AG" (id 5) (at 187.96 76.2 0)
+    (property "LCSC" "C503061" (id 4) (at 187.96 76.2 0)
+      (effects (font (size 1.27 1.27)) hide)
+    )
+    (property "MPN" "NCEP068N10G" (id 5) (at 187.96 76.2 0)
       (effects (font (size 1.27 1.27)) hide)
     )
@@
       (effects (font (size 1.27 1.27)) hide)
     )
-    (property "LCSC" "C500738" (id 4) (at 152.4 139.7 0)
-      (effects (font (size 1.27 1.27)) hide)
-    )
-    (property "MPN" "4m 1% 2W" (id 5) (at 152.4 139.7 0)
+    (property "LCSC" "C2904236" (id 4) (at 152.4 139.7 0)
+      (effects (font (size 1.27 1.27)) hide)
+    )
+    (property "MPN" "HoJLR2512-3W-4mR-1%" (id 5) (at 152.4 139.7 0)
       (effects (font (size 1.27 1.27)) hide)
     )
@@
       (effects (font (size 1.27 1.27)) hide)
     )
-    (property "LCSC" "" (id 4) (at 330.2 167.64 0)
+    (property "LCSC" "C441204" (id 4) (at 330.2 167.64 0)
       (effects (font (size 1.27 1.27)) hide)
     )
@@
       (effects (font (size 1.27 1.27)) hide)
     )
-    (property "LCSC" "C25744" (id 4) (at 104.14 86.36 0)
+    (property "LCSC" "C2906861" (id 4) (at 104.14 86.36 0)
       (effects (font (size 1.27 1.27)) hide)
     )
@@
       (effects (font (size 1.27 1.27)) hide)
     )
-    (property "LCSC" "C25744" (id 4) (at 104.14 124.46 0)
+    (property "LCSC" "C2906861" (id 4) (at 104.14 124.46 0)
       (effects (font (size 1.27 1.27)) hide)
     )
@@
       (effects (font (size 1.27 1.27)) hide)
     )
-    (property "LCSC" "C25744" (id 4) (at 30.48 116.84 0)
+    (property "LCSC" "C2906861" (id 4) (at 30.48 116.84 0)
       (effects (font (size 1.27 1.27)) hide)
     )
@@
       (effects (font (size 1.27 1.27)) hide)
     )
-    (property "LCSC" "C25744" (id 4) (at 38.1 116.84 0)
+    (property "LCSC" "C2906861" (id 4) (at 38.1 116.84 0)
       (effects (font (size 1.27 1.27)) hide)
     )
@@
       (effects (font (size 1.27 1.27)) hide)
     )
-    (property "LCSC" "C25744" (id 4) (at 200.66 86.36 0)
+    (property "LCSC" "C2906861" (id 4) (at 200.66 86.36 0)
       (effects (font (size 1.27 1.27)) hide)
     )
@@
       (effects (font (size 1.27 1.27)) hide)
     )
-    (property "LCSC" "C25744" (id 4) (at 200.66 124.46 0)
+    (property "LCSC" "C2906861" (id 4) (at 200.66 124.46 0)
       (effects (font (size 1.27 1.27)) hide)
     )
@@
       (effects (font (size 1.27 1.27)) hide)
     )
-    (property "LCSC" "C25744" (id 4) (at 276.86 116.84 0)
+    (property "LCSC" "C2906861" (id 4) (at 276.86 116.84 0)
       (effects (font (size 1.27 1.27)) hide)
     )
@@
       (effects (font (size 1.27 1.27)) hide)
     )
-    (property "LCSC" "C25744" (id 4) (at 284.48 116.84 0)
-      (effects (font (size 1.27 1.27)) hide)
-    )
+    (property "LCSC" "C2906861" (id 4) (at 284.48 116.84 0)
+      (effects (font (size 1.27 1.27)) hide)
+    )
