File: 01_hardware/kicad_project/sbb.kicad_sch (KiCad schematic)
At the start: 48 parts, among them J2 VOUT 1.5-48V, Q1 NCEP0140AG, Q2 NCEP068N10G, Q3 NCEP068N10G, Q4 NCEP0140AG, U2 UCC27211DDAR, U3 UCC27211DDAR

Commit message: Rev E2: debug-port series resistors, DRC clean (0 errors / 0 warnings)
- R123-R128 47.5 Ohm 0402 (C82290) in SWDIO, SWCLK, TP_DAC, TP_GPIO1,
  TP_GPIO2, NRST; R129 2 Ohm 0603 (C2933191) +3V3 -> J6.7 / J7 VTref
  (PROG_3V3). Placed on the MCU side of the J6/J7 branch, inserted into
  the existing traces.
- Cleared the 16 courtyard overlaps (T1/CR*/R64, T2/D8/C94/R116/C95/Q11/
  R114, C98/R122, C69/U11, C34/U1) with small moves, tracks re-attached;
  silk warnings gone. Parity 291 parts / 796 pads, 0 mismatches.
- BOMs, JLC BOM/CPL, gerbers, PDFs, EasyEDA zip, sourcing workbook,
  design notes, DRC report, README updated; scripts in 04_scripts/pcb6.

Co-Authored-By: Claude Opus 5.5 <noreply@anthropic.com>
Claude-Session: https://claude.ai/code/session_01A35wrnwFKLPSaRSxxHs471
Changed lines of the file:
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@@
   (symbol (lib_id "Transistor_FET:BSC040N10NS5") (at 116.84 114.3 0) (unit 1)
     (in_bom yes) (on_board yes)
-    (property "Reference" "Q2" (id 0) (at 112.712 109.89 0)
+    (property "Reference" "Q2" (id 0) (at 123.203 113.284 0)
       (effects (font (size 1.27 1.27)))
     )
-    (property "Value" "NCEP068N10G" (id 1) (at 112.712 118.71 0)
+    (property "Value" "NCEP068N10G" (id 1) (at 128.461 115.316 0)
       (effects (font (size 1.27 1.27)))
     )
@@
   (symbol (lib_id "Transistor_FET:BSC040N10NS5") (at 187.96 76.2 0) (mirror y) (unit 1)
     (in_bom yes) (on_board yes)
-    (property "Reference" "Q3" (id 0) (at 192.088 69.758 0)
+    (property "Reference" "Q3" (id 0) (at 181.597 75.184 0)
       (effects (font (size 1.27 1.27)))
     )
-    (property "Value" "NCEP068N10G" (id 1) (at 192.088 71.79 0)
+    (property "Value" "NCEP068N10G" (id 1) (at 176.339 77.216 0)
       (effects (font (size 1.27 1.27)))
     )
