File: 01_hardware/kicad_project/sec_aux.kicad_sch (KiCad schematic)
At the start: 18 parts, among them U4 LMR16006XDDCR, U5 AMS1117-5.0

Commit message: update D
Parts:
- added TP10: GND, TestPoint:TestPoint_Pad_D1.5mm, symbol Connector:TestPoint
- added TP5: VBUS, TestPoint:TestPoint_Pad_D1.5mm, symbol Connector:TestPoint
- added TP6: +10V, TestPoint:TestPoint_Pad_D1.5mm, symbol Connector:TestPoint
- added TP7: +5V, TestPoint:TestPoint_Pad_D1.5mm, symbol Connector:TestPoint
- added TP8: +3V3, TestPoint:TestPoint_Pad_D1.5mm, symbol Connector:TestPoint
- added TP9: +3V3A, TestPoint:TestPoint_Pad_D1.5mm, symbol Connector:TestPoint
- D2: value B1100 -> SS110; footprint Diode_SMD:D_SOD-123F -> Diode_SMD:D_SMA; LCSC (none) -> C224219; MPN B1100 / SS110 -> SS110
Connections:
- net +10V: now also TP6.1
- net +3V3: now also TP8.1
- net +3V3A: now also TP9.1
- net +5V: now also TP7.1
- net GND: now also TP10.1
- net VBUS: now also TP5.1
