File: 01_hardware/kicad_project/sec_aux.kicad_sch (KiCad schematic)
At the start: 24 parts, among them U4 LMR16006XDDCR, U5 AMS1117-5.0

Commit message: Rev D order prep: common F1/L2/L3 parts, JLC-checked LCSC numbers, assembly files
- F1: 2512 -> 1206 7 A 63 V fuse (Littelfuse 0458007.DR, C206980; 2nd source Schurter 3413.0326.11)
- L2/L3: SRP5030 -> 5040 shielded 47 uH (SWPA5040S470MT, C86617; 2nd source SRN5040-470M, NRS5040T470MMGK)
- EN_AUX re-routed off the L2 pad gap; VIN track centred between the L3 pads (0.4 mm each side)
- LCSC numbers checked in the JLCPCB library for every assembled part (design.py JLC_LCSC),
  written to the BOMs, schematic and PCB fields
- New JLC assembly upload files DCDC_JLC_BOM.csv / DCDC_JLC_CPL.csv (217 parts; U1, T1,
  connectors, headers and SW1 hand-soldered) and jlc_order_files.py to rebuild them
- 03_calculations/aux_fuse_check.py: aux inductor peak 0.27 A vs 1.1 A Isat; F1 4.8 A at 12 V / 50 W
- Design notes (docx/pdf), README, Gerbers, CPL, PDFs and DRC report regenerated
- Checks: DRC (JLC rules) 0 errors / 0 unconnected, netlist 134 nets / 257 parts 0 errors,
  isolation check 0 errors, silkscreen clean

Co-Authored-By: Claude Opus 5.5 <noreply@anthropic.com>
Claude-Session: https://claude.ai/code/session_01A35wrnwFKLPSaRSxxHs471
Parts:
- C21: LCSC (none) -> C153036
- C22: LCSC (none) -> C88219
- C23: LCSC (none) -> C307331
- C24, C25, C26: LCSC (none) -> C15850
- C27: LCSC (none) -> C45783
- C28: LCSC (none) -> C52923
- C29: LCSC (none) -> C1525
- FB1: LCSC (none) -> C1002
- L2: footprint Inductor_SMD:L_Bourns_SRP5030T -> Inductor_SMD:L_Sunlord_SWPA5040S; LCSC (none) -> C86617; MPN 47u 1A -> SWPA5040S470MT
- R16: LCSC (none) -> C23178
- R17: LCSC (none) -> C36871
- R18: LCSC (none) -> C25750
- R19: LCSC (none) -> C25744
Changed lines of the file:
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@@
       (effects (font (size 1.27 1.27)) hide)
     )
-    (property "LCSC" "" (id 4) (at 40.64 83.82 0)
+    (property "LCSC" "C153036" (id 4) (at 40.64 83.82 0)
       (effects (font (size 1.27 1.27)) hide)
     )
@@
       (effects (font (size 1.27 1.27)) hide)
     )
-    (property "LCSC" "" (id 4) (at 22.86 83.82 0)
+    (property "LCSC" "C88219" (id 4) (at 22.86 83.82 0)
       (effects (font (size 1.27 1.27)) hide)
     )
@@
       (effects (font (size 1.27 1.27)) hide)
     )
-    (property "LCSC" "" (id 4) (at 58.42 81.28 0)
+    (property "LCSC" "C23178" (id 4) (at 58.42 81.28 0)
       (effects (font (size 1.27 1.27)) hide)
     )
@@
       (effects (font (size 1.27 1.27)) hide)
     )
-    (property "LCSC" "" (id 4) (at 58.42 96.52 0)
+    (property "LCSC" "C36871" (id 4) (at 58.42 96.52 0)
       (effects (font (size 1.27 1.27)) hide)
     )
@@
       (effects (font (size 1.27 1.27)) hide)
     )
-    (property "LCSC" "" (id 4) (at 109.22 76.2 0)
+    (property "LCSC" "C307331" (id 4) (at 109.22 76.2 0)
       (effects (font (size 1.27 1.27)) hide)
     )
@@
       (effects (font (size 1.0 1.0)))
     )
-    (property "Footprint" "Inductor_SMD:L_Bourns_SRP5030T" (id 2) (at 129.54 83.82 0)
+    (property "Footprint" "Inductor_SMD:L_Sunlord_SWPA5040S" (id 2) (at 129.54 83.82 0)
       (effects (font (size 1.27 1.27)) hide)
     )
@@
       (effects (font (size 1.27 1.27)) hide)
     )
-    (property "LCSC" "" (id 4) (at 129.54 83.82 0)
-      (effects (font (size 1.27 1.27)) hide)
-    )
-    (property "MPN" "47u 1A" (id 5) (at 129.54 83.82 0)
+    (property "LCSC" "C86617" (id 4) (at 129.54 83.82 0)
+      (effects (font (size 1.27 1.27)) hide)
+    )
+    (property "MPN" "SWPA5040S470MT" (id 5) (at 129.54 83.82 0)
       (effects (font (size 1.27 1.27)) hide)
     )
@@
       (effects (font (size 1.27 1.27)) hide)
     )
-    (property "LCSC" "" (id 4) (at 144.78 93.98 0)
+    (property "LCSC" "C25750" (id 4) (at 144.78 93.98 0)
       (effects (font (size 1.27 1.27)) hide)
     )
@@
       (effects (font (size 1.27 1.27)) hide)
     )
-    (property "LCSC" "" (id 4) (at 144.78 109.22 0)
+    (property "LCSC" "C25744" (id 4) (at 144.78 109.22 0)
       (effects (font (size 1.27 1.27)) hide)
     )
@@
       (effects (font (size 1.27 1.27)) hide)
     )
-    (property "LCSC" "" (id 4) (at 154.94 93.98 0)
+    (property "LCSC" "C15850" (id 4) (at 154.94 93.98 0)
       (effects (font (size 1.27 1.27)) hide)
     )
@@
       (effects (font (size 1.27 1.27)) hide)
     )
-    (property "LCSC" "" (id 4) (at 167.64 93.98 0)
+    (property "LCSC" "C15850" (id 4) (at 167.64 93.98 0)
       (effects (font (size 1.27 1.27)) hide)
     )
@@
       (effects (font (size 1.27 1.27)) hide)
     )
-    (property "LCSC" "" (id 4) (at 208.28 93.98 0)
+    (property "LCSC" "C15850" (id 4) (at 208.28 93.98 0)
       (effects (font (size 1.27 1.27)) hide)
     )
@@
       (effects (font (size 1.27 1.27)) hide)
     )
-    (property "LCSC" "" (id 4) (at 236.22 93.98 0)
+    (property "LCSC" "C45783" (id 4) (at 236.22 93.98 0)
       (effects (font (size 1.27 1.27)) hide)
     )
@@
       (effects (font (size 1.27 1.27)) hide)
     )
-    (property "LCSC" "" (id 4) (at 251.46 83.82 0)
+    (property "LCSC" "C1002" (id 4) (at 251.46 83.82 0)
       (effects (font (size 1.27 1.27)) hide)
     )
@@
       (effects (font (size 1.27 1.27)) hide)
     )
-    (property "LCSC" "" (id 4) (at 266.7 93.98 0)
+    (property "LCSC" "C52923" (id 4) (at 266.7 93.98 0)
       (effects (font (size 1.27 1.27)) hide)
     )
@@
       (effects (font (size 1.27 1.27)) hide)
     )
-    (property "LCSC" "" (id 4) (at 279.4 93.98 0)
-      (effects (font (size 1.27 1.27)) hide)
-    )
+    (property "LCSC" "C1525" (id 4) (at 279.4 93.98 0)
+      (effects (font (size 1.27 1.27)) hide)
+    )

Commit message: Rev E: isolated flyback aux supply, VREF+ back to 3.3 V, 1 oz re-layout
- New isolated aux flyback (sheet iso_pwr): UC3843B U20 from +10V_P, FDN86246 Q11,
  PA3855.006NLT EP13 T2, SS110 D9 -> isolated +10 V; secondary regulation TL431 U22 +
  EL357N opto U21 into COMP; RCD clamp D8/R116/C94; 2 A primary limit (R114)
- Secondary rails from the flyback, not VBUS: +10 V -> U4 10->5 V -> U5 TLV75533 3.3 V;
  MCU, CAN and drivers up before the LLC starts
- U12 -> CA-IS3742LW (data only); REF3030 U19 removed, VREF+ = +3V3A (3.3 V full scale)
- PCB re-placed / re-routed for 1 oz outer / 0.5 oz inner: power pours on F.Cu, In1 solid
  ground planes, gate loops as tight HO/HS pairs, 1.7 mm power-via pitch, per-pad GND vias
  in the MCU area; copper loss ~0.5 W at 50 W (03_calculations/copper_check.txt)
- DRC (JLC rules) 0 errors / 0 unconnected; netlist 148 nets / 284 parts 0 errors;
  isolation bands clear; BOM / JLC BOM+CPL / Gerbers / PDFs / design notes / READMEs updated
- Scripts: 04_scripts/pcb5 (placement, pours, routing, floods, island vias, silk),
  03_calculations/flyback_aux.py, copper_check.py

Co-Authored-By: Claude Opus 5.5 <noreply@anthropic.com>
Claude-Session: https://claude.ai/code/session_01A35wrnwFKLPSaRSxxHs471
Parts:
- removed TP5: VBUS, TestPoint:TestPoint_Pad_D1.5mm, symbol Connector:TestPoint
- removed U5: AMS1117-5.0, Package_TO_SOT_SMD:SOT-223-3_TabPin2, symbol Regulator_Linear:AMS1117-5.0
- added C86: 1u 10V, Capacitor_SMD:C_0402_1005Metric, symbol Device:C
- added U5: TLV75533PDBVR, Package_TO_SOT_SMD:SOT-23-5, symbol Regulator_Linear:TLV75533PDBV
- C21: value 2.2u 100V X7R -> 10u 25V X5R; footprint Capacitor_SMD:C_1210_3225Metric -> Capacitor_SMD:C_0805_2012Metric; LCSC C153036 -> C15850; MPN 2.2u 100V X7R -> 10u 25V X5R
- C22: value 100n 100V -> 100n 25V; footprint Capacitor_SMD:C_0603_1608Metric -> Capacitor_SMD:C_0402_1005Metric; LCSC C88219 -> C307331; MPN 100n 100V -> 100n 25V
- R16: value 470k -> 56k 1%; footprint Resistor_SMD:R_0603_1608Metric -> Resistor_SMD:R_0402_1005Metric; LCSC C23178 -> C25796; MPN 470k -> 56k 1%
- R17: value 68k -> 15k 1%; LCSC C36871 -> C25756; MPN 68k -> 15k 1%
- R18: value 120k 1% -> 56k 1%; LCSC C25750 -> C25796; MPN 120k 1% -> 56k 1%
Connections:
- net VBUS is gone; now on net +10V: C21.1, C22.1, R16.1, U4.5 (VIN)
- net +10V: no longer L2.2, R18.1
- net +3V3: now also U5.5 (OUT)
- net +5V: now also L2.2, R18.1, C86.1, U5.1 (IN), U5.3 (EN)
- net GND: now also C86.2, U5.2 (GND)
- no-connect marks 0 -> 1

Commit message: Rev E BOM: in-stock LCSC first source for every part; 2nd/3rd sources checked
- First sources swapped (same footprints, layout unchanged): U1 STM32G474RBT3,
  Q2/Q3/Q5/Q6 NCEP068N10G, 10k 0402 FOJAN, 100n 0402 merged onto C307331,
  1u 0402 CCTC, R62/R63/R89/R82, FB1 Murata BLM18KG601SN1D, L2/L3 cjiang
  FNR5040S470MT, C82 KEMET C0G (was X7R), RS1 Milliohm HoJLR2512, SS110 MDD
- LCSC part numbers for the hand-soldered headers (J1-J5, J7, JP1)
- Schematic and PCB fields, BOM, JLC BOM/CPL, PDFs and design notes regenerated;
  netlist check 0 errors, DRC unchanged
- BOM_sourcing_revE.xlsx: live LCSC stock 2026-10-20, 2nd/3rd sources checked
  for pinout / land pattern / ratings, PCB reserve options for T2 and U9

Co-Authored-By: Claude Opus 5.5 <noreply@anthropic.com>
Claude-Session: https://claude.ai/code/session_01A35wrnwFKLPSaRSxxHs471
Parts:
- C28, C86: LCSC C52923 -> C20539426
- C29: LCSC C1525 -> C307331
- D2: LCSC C224219 -> C2482
- FB1: LCSC C1002 -> C85833; MPN 600R@100MHz -> BLM18KG601SN1D
- L2: LCSC C86617 -> C167974; MPN SWPA5040S470MT -> FNR5040S470MT
- R19: LCSC C25744 -> C2906861
Changed lines of the file:
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@@
       (effects (font (size 1.27 1.27)) hide)
     )
-    (property "LCSC" "C224219" (id 4) (at 114.3 96.52 0)
+    (property "LCSC" "C2482" (id 4) (at 114.3 96.52 0)
       (effects (font (size 1.27 1.27)) hide)
     )
@@
       (effects (font (size 1.27 1.27)) hide)
     )
-    (property "LCSC" "C86617" (id 4) (at 129.54 83.82 0)
-      (effects (font (size 1.27 1.27)) hide)
-    )
-    (property "MPN" "SWPA5040S470MT" (id 5) (at 129.54 83.82 0)
+    (property "LCSC" "C167974" (id 4) (at 129.54 83.82 0)
+      (effects (font (size 1.27 1.27)) hide)
+    )
+    (property "MPN" "FNR5040S470MT" (id 5) (at 129.54 83.82 0)
       (effects (font (size 1.27 1.27)) hide)
     )
@@
       (effects (font (size 1.27 1.27)) hide)
     )
-    (property "LCSC" "C25744" (id 4) (at 144.78 109.22 0)
+    (property "LCSC" "C2906861" (id 4) (at 144.78 109.22 0)
       (effects (font (size 1.27 1.27)) hide)
     )
@@
       (effects (font (size 1.27 1.27)) hide)
     )
-    (property "LCSC" "C52923" (id 4) (at 220.98 93.98 0)
+    (property "LCSC" "C20539426" (id 4) (at 220.98 93.98 0)
       (effects (font (size 1.27 1.27)) hide)
     )
@@
       (effects (font (size 1.27 1.27)) hide)
     )
-    (property "LCSC" "C1002" (id 4) (at 251.46 83.82 0)
-      (effects (font (size 1.27 1.27)) hide)
-    )
-    (property "MPN" "600R@100MHz" (id 5) (at 251.46 83.82 0)
+    (property "LCSC" "C85833" (id 4) (at 251.46 83.82 0)
+      (effects (font (size 1.27 1.27)) hide)
+    )
+    (property "MPN" "BLM18KG601SN1D" (id 5) (at 251.46 83.82 0)
       (effects (font (size 1.27 1.27)) hide)
     )
@@
       (effects (font (size 1.27 1.27)) hide)
     )
-    (property "LCSC" "C52923" (id 4) (at 266.7 93.98 0)
+    (property "LCSC" "C20539426" (id 4) (at 266.7 93.98 0)
       (effects (font (size 1.27 1.27)) hide)
     )
@@
       (effects (font (size 1.27 1.27)) hide)
     )
-    (property "LCSC" "C1525" (id 4) (at 279.4 93.98 0)
-      (effects (font (size 1.27 1.27)) hide)
-    )
+    (property "LCSC" "C307331" (id 4) (at 279.4 93.98 0)
+      (effects (font (size 1.27 1.27)) hide)
+    )
