File: 01_hardware/kicad_project/sense.kicad_sch (KiCad schematic)
At the start: 20 parts, among them U7 INA181A1IDBVR, U8 INA181A2IDBVR

Commit message: update D
Parts:
- added TP13: IL_SNS, TestPoint:TestPoint_Pad_D1.5mm, symbol Connector:TestPoint
- added TP14: IOUT_SNS, TestPoint:TestPoint_Pad_D1.5mm, symbol Connector:TestPoint
Connections:
- net IL_SNS: now also TP13.1
- net IOUT_SNS: now also TP14.1
