File: 01_hardware/kicad_project/DCDC_LLC_4SBB_G474.kicad_pcb (KiCad board)
At the start: 4 copper layers, 160 x 105 mm, 197 parts, among them J1 VIN 12-48V, J2 VOUT 1.5-48V, J3 CAN A, J4 CAN B, J5 ADDR HDR, J6 PROG PADS, J7 ARM SWD 10, Q1 NCEP0140AG, Q2 NCEP0160AG, Q3 NCEP0160AG, Q4 NCEP0140AG, Q5 NCEP0160AG, Q6 NCEP0160AG, Q7 BSC160N15NS5, Q8 BSC160N15NS5, SW1 DIP-6, T1 PQ2620 4:8+8, U1 STM32G474RBT6, U10 UCC27211DDAR, U11 UCC27524DR, U12 CA-IS3642LVW, U13 LMR16006XDDCR, U14 AMS1117-5.0, U2 UCC27211DDAR, U3 UCC27211DDAR, U4 LMR16006XDDCR, U5 AMS1117-5.0, U7 INA181A1IDBVR, U8 INA181A2IDBVR, U9 CA-IS3062VW, Y1 8MHz 12pF

Commit message: update D
Parts:
- added C79: 1n C0G, Capacitor_SMD:C_0402_1005Metric, F.Cu at (53.5, 76.6)
- added C80: 100n, Capacitor_SMD:C_0402_1005Metric, F.Cu at (60.0, 75.4)
- added R100: 10k, Resistor_SMD:R_0402_1005Metric, F.Cu at (113.2, 71.9)
- added R101: 10k, Resistor_SMD:R_0402_1005Metric, F.Cu at (111.2, 71.9)
- added R102: 10k, Resistor_SMD:R_0402_1005Metric, F.Cu at (103.9, 78.3)
- added R103: 10k, Resistor_SMD:R_0402_1005Metric, F.Cu at (103.9, 80.0)
- added R104: 10k, Resistor_SMD:R_0402_1005Metric, F.Cu at (103.9, 81.5)
- added R105: 10k, Resistor_SMD:R_0402_1005Metric, F.Cu at (103.9, 83.2)
- added R81: 191k 1%, Resistor_SMD:R_1206_3216Metric, F.Cu at (56.3, 74.6)
- added R82: 10k 1%, Resistor_SMD:R_0402_1005Metric, F.Cu at (54.8, 79.8)
- added R83: 10k, Resistor_SMD:R_0402_1005Metric, F.Cu at (61.5, 72.1)
- added R84: 2.2M, Resistor_SMD:R_0402_1005Metric, F.Cu at (59.1, 73.0)
- added R85: 1k, Resistor_SMD:R_0402_1005Metric, F.Cu at (57.0, 79.3)
- added R90: 10k, Resistor_SMD:R_0402_1005Metric, F.Cu at (104.7, 90.1)
- added R91: 10k, Resistor_SMD:R_0402_1005Metric, F.Cu at (106.2, 90.1)
- added R92: 10k, Resistor_SMD:R_0402_1005Metric, F.Cu at (107.8, 90.1)
- added R93: 10k, Resistor_SMD:R_0402_1005Metric, F.Cu at (115.8, 90.1)
- added R94: 10k, Resistor_SMD:R_0402_1005Metric, F.Cu at (122.1, 85.5)
- added R95: 10k, Resistor_SMD:R_0402_1005Metric, F.Cu at (122.1, 83.9)
- added R96: 10k, Resistor_SMD:R_0402_1005Metric, F.Cu at (122.1, 82.3)
- added R97: 10k, Resistor_SMD:R_0402_1005Metric, F.Cu at (122.1, 80.2)
- added R98: 10k, Resistor_SMD:R_0402_1005Metric, F.Cu at (122.1, 78.2)
- added R99: 10k, Resistor_SMD:R_0402_1005Metric, F.Cu at (114.8, 71.9)
- added TP1: VIN, TestPoint:TestPoint_Pad_D1.5mm, F.Cu at (21.0, 13.8)
- added TP10: GND, TestPoint:TestPoint_Pad_D1.5mm, F.Cu at (78.5, 69.0)
- added TP11: VOUT, TestPoint:TestPoint_Pad_D1.5mm, F.Cu at (152.3, 42.3)
- added TP12: GND, TestPoint:TestPoint_Pad_D1.5mm, F.Cu at (132.6, 54.5)
- added TP13: IL_SNS, TestPoint:TestPoint_Pad_D1.5mm, F.Cu at (120.1, 51.6)
- added TP14: IOUT_SNS, TestPoint:TestPoint_Pad_D1.5mm, F.Cu at (132.8, 58.6)
- added TP15: VIN_OVP, TestPoint:TestPoint_Pad_D1.5mm, F.Cu at (82.4, 80.7)
- added TP2: GNDP, TestPoint:TestPoint_Pad_D1.5mm, F.Cu at (39.2, 47.0)
- added TP3: +10V_P, TestPoint:TestPoint_Pad_D1.5mm, F.Cu at (33.6, 73.3)
- added TP4: +5V_P, TestPoint:TestPoint_Pad_D1.5mm, F.Cu at (42.2, 75.8)
- added TP5: VBUS, TestPoint:TestPoint_Pad_D1.5mm, F.Cu at (95.4, 48.0)
- added TP6: +10V, TestPoint:TestPoint_Pad_D1.5mm, F.Cu at (86.1, 63.6)
- added TP7: +5V, TestPoint:TestPoint_Pad_D1.5mm, F.Cu at (96.2, 72.8)
- added TP8: +3V3, TestPoint:TestPoint_Pad_D1.5mm, F.Cu at (74.1, 67.1)
- added TP9: +3V3A, TestPoint:TestPoint_Pad_D1.5mm, F.Cu at (128.3, 76.4)
- added U15: LMV331IDBVR, Package_TO_SOT_SMD:SOT-23-5, F.Cu at (60.5, 78.8)
- added U16: TL431AIDBZR, Package_TO_SOT_SMD:SOT-23, F.Cu at (59.2, 83.7)
- C38, C39: value 18p C0G -> 12p C0G
- D2, D6: value B1100 -> SS110; footprint Diode_SMD:D_SOD-123F -> Diode_SMD:D_SMA
- Y1: value 8MHz 12pF -> 16MHz 9pF
- moved TH1 54.9 mm to (114.0, 38.8), turned to 90 degrees
- moved C48 45.5 mm to (116.3, 48.9), turned to 0 degrees
- moved R29 45.0 mm to (115.2, 46.5)
- moved C4 31.4 mm to (88.5, 32.8), turned to 0 degrees
- moved C12 31.0 mm to (156.8, 23.0), turned to -90 degrees
- moved R1 29.2 mm to (141.7, 57.1), turned to 0 degrees
- moved J2 28.0 mm to (148.0, 54.0)
- moved C3 25.1 mm to (88.5, 29.5)
- moved C39 22.6 mm to (116.0, 92.9)
- moved C35 21.6 mm to (122.8, 89.0), turned to 90 degrees
- moved C40 20.9 mm to (112.7, 94.7), turned to 0 degrees
- moved R64 20.4 mm to (48.6, 20.3)
- moved C67 19.0 mm to (49.5, 25.6)
- moved C8 18.8 mm to (146.9, 23.0), turned to -90 degrees
- moved C2 18.7 mm to (88.5, 26.2)
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Connections:
- U1 pad 14: (no net) -> SP_PA2
- U1 pad 17: (no net) -> SP_PA3
- U1 pad 18: NTC_SNS -> SP_PA4
- U1 pad 2: (no net) -> SP_PC13
- U1 pad 20: (no net) -> NTC_SNS
- U1 pad 21: (no net) -> SP_PA7
- U1 pad 26: (no net) -> SP_PB2
- U1 pad 3: (no net) -> SP_PC14
- U1 pad 30: (no net) -> SP_PB10
- U1 pad 38: (no net) -> SP_PC6
- U1 pad 39: (no net) -> SP_PC7
- U1 pad 4: (no net) -> SP_PC15
- U1 pad 44: (no net) -> SP_PA10
- U1 pad 51: (no net) -> VIN_OVP
- U1 pad 54: (no net) -> SP_PC12
- U1 pad 55: (no net) -> SP_PD2
- U1 pad 57: (no net) -> SP_PB4
- U1 pad 58: (no net) -> SP_PB5
- U12 pad 14: (no net) -> VIN_OVP
- U12 pad 3: GNDP -> OVP_P
Routing:
- net GND: track 137.5 -> 309.8 mm, vias 98 -> 181
- net GNDP: track 40.1 -> 108.8 mm, vias 29 -> 58
- net VOUT_N: track 76.0 -> 20.9 mm, vias 1 -> 2
- net PGND: track 181.9 -> 135.6 mm, vias 5 -> 8
- net HB_SW: track 95.1 -> 50.8 mm, vias 1 -> 2
- net +3V3: track 217.0 -> 256.6 mm, vias 9 -> 11
- net VIN_OVP: track 0.00 -> 37.5 mm
- net VIN: track 159.0 -> 196.0 mm, vias 5 -> 4
- net NTC_SNS: track 16.3 -> 49.6 mm, vias 0 -> 2
- net SW1: track 85.8 -> 53.8 mm, vias 3 -> 2
- net +3V3A: track 75.2 -> 101.8 mm, vias 2 -> 5
- net G3: track 50.6 -> 24.8 mm
- net VOUT: track 145.3 -> 121.1 mm, vias 2 -> 0
- net G7: track 34.9 -> 11.9 mm, vias 2 -> 3
- net ADDR4: track 34.2 -> 56.8 mm, vias 3 -> 2
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- added copper zone on F.Cu, net CR_MID
- added copper zone on B.Cu, net GND
- added copper zone on F.Cu, net GND
- added copper zone on In2.Cu, net GND
- added copper zone on B.Cu, net GNDP
- added copper zone on F.Cu, net GNDP
- added copper zone on In2.Cu, net GNDP
- added copper zone on B.Cu, net GND_ISO
- added copper zone on F.Cu, net GND_ISO
- added copper zone on In2.Cu, net GND_ISO
- added copper zone on F.Cu, net HB_SW
- added copper zone on F.Cu, net PGND
- added copper zone on F.Cu, net SR_D1
- added copper zone on F.Cu, net SR_D2
- added copper zone on F.Cu, net SW1
- added copper zone on F.Cu, net SW2
- added copper zone on F.Cu, net VBUS
- added copper zone on F.Cu, net VIN
- added copper zone on F.Cu, net VOUT

Commit message: update
Parts:
- C1, C11, C60: value 47u 63V -> 47u
- C56: value 2.2n 2kV DNP -> 2.2n
- C66: value 1n Y1 DNP -> 1n
- CR1, CR2, CR3, CR4, CR5, CR6: value 100n 100V C0G -> 100n
- J1: value VIN 12-48V -> VIN
- J2: value VOUT 1.5-48V -> VOUT
- J3: value CAN A -> CAN
- J4: value CAN B -> CAN
- J5: value ADDR HDR -> ADDR
- J6: value PROG PADS -> PROG
- J7: value ARM SWD 10 -> SWD
- L1: value 22u 23A sat -> 22u
- L2, L3: value 47u 1A -> 47u
- RS1: value 4m 1% 2W -> 4m
- RSH1: value 10m 1% 1W -> 10m
- T1: value PQ2620 4:8+8 -> PQ2620
- Y1: value 16MHz 9pF -> 16MHz

Commit message: add CAN termination res jumper
Parts:
- JP1: footprint Connector_PinHeader_2.54mm:PinHeader_1x02_P2.54mm_Vertical -> PinHeader_2x02_P2.54mm_Vertical
Connections:
- JP1 pad 1: CAN_TL -> CAN_TH
- JP1 pad 2: CANL -> CANH
- R30 pad 1: CANH -> CAN_TH
Routing:
- net CAN_TH: track 0.00 -> 7.63 mm
- net CAN_TL: track 9.67 -> 12.8 mm
- net CANL: track 46.9 -> 49.2 mm
- net CANH: track 50.0 -> 48.2 mm
Other:
- board text added: "TERM 1-2+3-4"

Commit message: update silkscreen
Parts:
- moved JP1 5.08 mm to (146.9, 94.7)
Routing:
- net CANL: track 49.2 -> 58.6 mm
- net CAN_TH: track 7.63 -> 12.7 mm
- net CANH: track 48.2 -> 53.3 mm
- net CAN_TL: track 12.8 -> 17.9 mm
Other:
- board text added: "1"
- board text added: "CAN TERM"
- board text added: "CAN_GND"
- board text added: "CAN_H"
- board text added: "CAN_L"
- board text added: "VIN+"
- board text added: "VIN-"
- board text added: "VOUT+"
- board text added: "VOUT-"
- board text removed: "TERM 1-2+3-4"
