File: 01_hardware/kicad_project/io.kicad_sch (KiCad schematic)
At the start: 24 parts, among them J5 ADDR HDR, J6 PROG PADS, J7 ARM SWD 10, SW1 DIP-6

Commit message: Rev D order prep: common F1/L2/L3 parts, JLC-checked LCSC numbers, assembly files
- F1: 2512 -> 1206 7 A 63 V fuse (Littelfuse 0458007.DR, C206980; 2nd source Schurter 3413.0326.11)
- L2/L3: SRP5030 -> 5040 shielded 47 uH (SWPA5040S470MT, C86617; 2nd source SRN5040-470M, NRS5040T470MMGK)
- EN_AUX re-routed off the L2 pad gap; VIN track centred between the L3 pads (0.4 mm each side)
- LCSC numbers checked in the JLCPCB library for every assembled part (design.py JLC_LCSC),
  written to the BOMs, schematic and PCB fields
- New JLC assembly upload files DCDC_JLC_BOM.csv / DCDC_JLC_CPL.csv (217 parts; U1, T1,
  connectors, headers and SW1 hand-soldered) and jlc_order_files.py to rebuild them
- 03_calculations/aux_fuse_check.py: aux inductor peak 0.27 A vs 1.1 A Isat; F1 4.8 A at 12 V / 50 W
- Design notes (docx/pdf), README, Gerbers, CPL, PDFs and DRC report regenerated
- Checks: DRC (JLC rules) 0 errors / 0 unconnected, netlist 134 nets / 257 parts 0 errors,
  isolation check 0 errors, silkscreen clean

Co-Authored-By: Claude Opus 5.5 <noreply@anthropic.com>
Claude-Session: https://claude.ai/code/session_01A35wrnwFKLPSaRSxxHs471
Parts:
- D4: LCSC (none) -> C12624
- D5: LCSC (none) -> C2286
- R32, R33, R34, R35, R36, R37: LCSC (none) -> C25744
- R38, R39, R40, R41, R42, R43, R44, R45: LCSC (none) -> C11702
Changed lines of the file:
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@@
       (effects (font (size 1.27 1.27)) hide)
     )
-    (property "LCSC" "" (id 4) (at 129.54 71.12 0)
+    (property "LCSC" "C25744" (id 4) (at 129.54 71.12 0)
       (effects (font (size 1.27 1.27)) hide)
     )
@@
       (effects (font (size 1.27 1.27)) hide)
     )
-    (property "LCSC" "" (id 4) (at 129.54 129.54 0)
+    (property "LCSC" "C11702" (id 4) (at 129.54 129.54 0)
       (effects (font (size 1.27 1.27)) hide)
     )
@@
       (effects (font (size 1.27 1.27)) hide)
     )
-    (property "LCSC" "" (id 4) (at 116.84 71.12 0)
+    (property "LCSC" "C25744" (id 4) (at 116.84 71.12 0)
       (effects (font (size 1.27 1.27)) hide)
     )
@@
       (effects (font (size 1.27 1.27)) hide)
     )
-    (property "LCSC" "" (id 4) (at 116.84 129.54 0)
+    (property "LCSC" "C11702" (id 4) (at 116.84 129.54 0)
       (effects (font (size 1.27 1.27)) hide)
     )
@@
       (effects (font (size 1.27 1.27)) hide)
     )
-    (property "LCSC" "" (id 4) (at 104.14 71.12 0)
+    (property "LCSC" "C25744" (id 4) (at 104.14 71.12 0)
       (effects (font (size 1.27 1.27)) hide)
     )
@@
       (effects (font (size 1.27 1.27)) hide)
     )
-    (property "LCSC" "" (id 4) (at 104.14 129.54 0)
+    (property "LCSC" "C11702" (id 4) (at 104.14 129.54 0)
       (effects (font (size 1.27 1.27)) hide)
     )
@@
       (effects (font (size 1.27 1.27)) hide)
     )
-    (property "LCSC" "" (id 4) (at 91.44 71.12 0)
+    (property "LCSC" "C25744" (id 4) (at 91.44 71.12 0)
       (effects (font (size 1.27 1.27)) hide)
     )
@@
       (effects (font (size 1.27 1.27)) hide)
     )
-    (property "LCSC" "" (id 4) (at 91.44 129.54 0)
+    (property "LCSC" "C11702" (id 4) (at 91.44 129.54 0)
       (effects (font (size 1.27 1.27)) hide)
     )
@@
       (effects (font (size 1.27 1.27)) hide)
     )
-    (property "LCSC" "" (id 4) (at 78.74 71.12 0)
+    (property "LCSC" "C25744" (id 4) (at 78.74 71.12 0)
       (effects (font (size 1.27 1.27)) hide)
     )
@@
       (effects (font (size 1.27 1.27)) hide)
     )
-    (property "LCSC" "" (id 4) (at 78.74 129.54 0)
+    (property "LCSC" "C11702" (id 4) (at 78.74 129.54 0)
       (effects (font (size 1.27 1.27)) hide)
     )
@@
       (effects (font (size 1.27 1.27)) hide)
     )
-    (property "LCSC" "" (id 4) (at 66.04 71.12 0)
+    (property "LCSC" "C25744" (id 4) (at 66.04 71.12 0)
       (effects (font (size 1.27 1.27)) hide)
     )
@@
       (effects (font (size 1.27 1.27)) hide)
     )
-    (property "LCSC" "" (id 4) (at 66.04 129.54 0)
+    (property "LCSC" "C11702" (id 4) (at 66.04 129.54 0)
       (effects (font (size 1.27 1.27)) hide)
     )
@@
       (effects (font (size 1.27 1.27)) hide)
     )
-    (property "LCSC" "" (id 4) (at 274.32 76.2 0)
+    (property "LCSC" "C12624" (id 4) (at 274.32 76.2 0)
       (effects (font (size 1.27 1.27)) hide)
     )
@@
       (effects (font (size 1.27 1.27)) hide)
     )
-    (property "LCSC" "" (id 4) (at 254.0 76.2 0)
+    (property "LCSC" "C11702" (id 4) (at 254.0 76.2 0)
       (effects (font (size 1.27 1.27)) hide)
     )
@@
       (effects (font (size 1.27 1.27)) hide)
     )
-    (property "LCSC" "" (id 4) (at 274.32 96.52 0)
+    (property "LCSC" "C2286" (id 4) (at 274.32 96.52 0)
       (effects (font (size 1.27 1.27)) hide)
     )
@@
       (effects (font (size 1.27 1.27)) hide)
     )
-    (property "LCSC" "" (id 4) (at 254.0 96.52 0)
-      (effects (font (size 1.27 1.27)) hide)
-    )
+    (property "LCSC" "C11702" (id 4) (at 254.0 96.52 0)
+      (effects (font (size 1.27 1.27)) hide)
+    )

Commit message: JLC assembly files: add SW1, merge duplicate LCSC lines, fix rotations
- SW1 DIP switch added to BOM/CPL (C6331172) and given an LCSC field in
  schematic and PCB
- BOM lines sharing an LCSC number are merged (JLC unselects duplicates)
- CPL rotations corrected against JLC pin-1 markers; NCEP0160AG (Q2/Q3/Q5/Q6)
  centroid offset 1.0 mm for the JLC model
- U1 hand-soldered (own sample); DNP snubbers/Y-caps left out of CPL
- U12 stays CA-IS3642LVW (pre-order); TI ISOW7842FDWER C2861496 is a
  pin-compatible alternative

Co-Authored-By: Claude Opus 5.5 <noreply@anthropic.com>
Claude-Session: https://claude.ai/code/session_01A35wrnwFKLPSaRSxxHs471
Parts:
- SW1: LCSC (none) -> C6331172
Changed lines of the file:
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@@
       (effects (font (size 1.27 1.27)) hide)
     )
-    (property "LCSC" "" (id 4) (at 165.1 101.6 0)
+    (property "LCSC" "C6331172" (id 4) (at 165.1 101.6 0)
       (effects (font (size 1.27 1.27)) hide)
     )
