File: 01_hardware/kicad_project/llc.kicad_sch (KiCad schematic)
At the start: 41 parts, among them J1 VIN 12-48V, Q5 NCEP0160AG, Q6 NCEP0160AG, Q7 BSC160N15NS5, Q8 BSC160N15NS5, T1 PQ2620 4:8+8, U10 UCC27211DDAR, U11 UCC27524DR

Commit message: Rev D order prep: common F1/L2/L3 parts, JLC-checked LCSC numbers, assembly files
- F1: 2512 -> 1206 7 A 63 V fuse (Littelfuse 0458007.DR, C206980; 2nd source Schurter 3413.0326.11)
- L2/L3: SRP5030 -> 5040 shielded 47 uH (SWPA5040S470MT, C86617; 2nd source SRN5040-470M, NRS5040T470MMGK)
- EN_AUX re-routed off the L2 pad gap; VIN track centred between the L3 pads (0.4 mm each side)
- LCSC numbers checked in the JLCPCB library for every assembled part (design.py JLC_LCSC),
  written to the BOMs, schematic and PCB fields
- New JLC assembly upload files DCDC_JLC_BOM.csv / DCDC_JLC_CPL.csv (217 parts; U1, T1,
  connectors, headers and SW1 hand-soldered) and jlc_order_files.py to rebuild them
- 03_calculations/aux_fuse_check.py: aux inductor peak 0.27 A vs 1.1 A Isat; F1 4.8 A at 12 V / 50 W
- Design notes (docx/pdf), README, Gerbers, CPL, PDFs and DRC report regenerated
- Checks: DRC (JLC rules) 0 errors / 0 unconnected, netlist 134 nets / 257 parts 0 errors,
  isolation check 0 errors, silkscreen clean

Co-Authored-By: Claude Opus 5.5 <noreply@anthropic.com>
Claude-Session: https://claude.ai/code/session_01A35wrnwFKLPSaRSxxHs471
Parts:
- C60: LCSC (none) -> C249664
- C61, C62, C63: LCSC (none) -> C153036
- C67: LCSC (none) -> C14663
- C68: LCSC (none) -> C15849
- CR1, CR2, CR3, CR4, CR5, CR6: LCSC (none) -> C2940749
- D1: LCSC (none) -> C20883337
- F1: value 7A -> 7A 63V; footprint Fuse:Fuse_2512_6332Metric -> Fuse:Fuse_1206_3216Metric; LCSC (none) -> C206980; MPN 7A -> 0458007.DR
- R62, R63: LCSC (none) -> C22939
- R64, R65, R66, R69, R70, R71, R72, R73: LCSC (none) -> C25744
- R68: LCSC (none) -> C23164
- U11: LCSC C465729 -> C15849
Changed lines of the file:
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@@
       (effects (font (size 1.27 1.27)))
     )
-    (property "Value" "7A" (id 1) (at 43.18 65.662 90)
-      (effects (font (size 1.0 1.0)))
-    )
-    (property "Footprint" "Fuse:Fuse_2512_6332Metric" (id 2) (at 43.18 63.5 0)
+    (property "Value" "7A 63V" (id 1) (at 43.18 65.662 90)
+      (effects (font (size 1.0 1.0)))
+    )
+    (property "Footprint" "Fuse:Fuse_1206_3216Metric" (id 2) (at 43.18 63.5 0)
       (effects (font (size 1.27 1.27)) hide)
     )
@@
       (effects (font (size 1.27 1.27)) hide)
     )
-    (property "LCSC" "" (id 4) (at 43.18 63.5 0)
-      (effects (font (size 1.27 1.27)) hide)
-    )
-    (property "MPN" "7A" (id 5) (at 43.18 63.5 0)
+    (property "LCSC" "C206980" (id 4) (at 43.18 63.5 0)
+      (effects (font (size 1.27 1.27)) hide)
+    )
+    (property "MPN" "0458007.DR" (id 5) (at 43.18 63.5 0)
       (effects (font (size 1.27 1.27)) hide)
     )
@@
       (effects (font (size 1.27 1.27)) hide)
     )
-    (property "LCSC" "" (id 4) (at 48.26 78.74 0)
+    (property "LCSC" "C20883337" (id 4) (at 48.26 78.74 0)
       (effects (font (size 1.27 1.27)) hide)
     )
@@
       (effects (font (size 1.27 1.27)) hide)
     )
-    (property "LCSC" "" (id 4) (at 58.42 78.74 0)
+    (property "LCSC" "C249664" (id 4) (at 58.42 78.74 0)
       (effects (font (size 1.27 1.27)) hide)
     )
@@
       (effects (font (size 1.27 1.27)) hide)
     )
-    (property "LCSC" "" (id 4) (at 76.2 78.74 0)
+    (property "LCSC" "C153036" (id 4) (at 76.2 78.74 0)
       (effects (font (size 1.27 1.27)) hide)
     )
@@
       (effects (font (size 1.27 1.27)) hide)
     )
-    (property "LCSC" "" (id 4) (at 93.98 78.74 0)
+    (property "LCSC" "C153036" (id 4) (at 93.98 78.74 0)
       (effects (font (size 1.27 1.27)) hide)
     )
@@
       (effects (font (size 1.27 1.27)) hide)
     )
-    (property "LCSC" "" (id 4) (at 111.76 78.74 0)
+    (property "LCSC" "C153036" (id 4) (at 111.76 78.74 0)
       (effects (font (size 1.27 1.27)) hide)
     )
@@
       (effects (font (size 1.27 1.27)) hide)
     )
-    (property "LCSC" "" (id 4) (at 157.48 101.6 0)
+    (property "LCSC" "C2940749" (id 4) (at 157.48 101.6 0)
       (effects (font (size 1.27 1.27)) hide)
     )
@@
       (effects (font (size 1.27 1.27)) hide)
     )
-    (property "LCSC" "" (id 4) (at 175.26 101.6 0)
+    (property "LCSC" "C2940749" (id 4) (at 175.26 101.6 0)
       (effects (font (size 1.27 1.27)) hide)
     )
@@
       (effects (font (size 1.27 1.27)) hide)
     )
-    (property "LCSC" "" (id 4) (at 193.04 101.6 0)
+    (property "LCSC" "C2940749" (id 4) (at 193.04 101.6 0)
       (effects (font (size 1.27 1.27)) hide)
     )
@@
       (effects (font (size 1.27 1.27)) hide)
     )
-    (property "LCSC" "" (id 4) (at 157.48 121.92 0)
+    (property "LCSC" "C2940749" (id 4) (at 157.48 121.92 0)
       (effects (font (size 1.27 1.27)) hide)
     )
@@
       (effects (font (size 1.27 1.27)) hide)
     )
-    (property "LCSC" "" (id 4) (at 175.26 121.92 0)
+    (property "LCSC" "C2940749" (id 4) (at 175.26 121.92 0)
       (effects (font (size 1.27 1.27)) hide)
     )
@@
       (effects (font (size 1.27 1.27)) hide)
     )
-    (property "LCSC" "" (id 4) (at 193.04 121.92 0)
+    (property "LCSC" "C2940749" (id 4) (at 193.04 121.92 0)
       (effects (font (size 1.27 1.27)) hide)
     )
@@
       (effects (font (size 1.27 1.27)) hide)
     )
-    (property "LCSC" "" (id 4) (at 106.68 104.14 0)
+    (property "LCSC" "C14663" (id 4) (at 106.68 104.14 0)
       (effects (font (size 1.27 1.27)) hide)
     )
@@
       (effects (font (size 1.27 1.27)) hide)
     )
-    (property "LCSC" "" (id 4) (at 66.04 104.14 0)
+    (property "LCSC" "C15849" (id 4) (at 66.04 104.14 0)
       (effects (font (size 1.27 1.27)) hide)
     )
@@
       (effects (font (size 1.27 1.27)) hide)
     )
-    (property "LCSC" "" (id 4) (at 121.92 63.5 0)
+    (property "LCSC" "C22939" (id 4) (at 121.92 63.5 0)
       (effects (font (size 1.27 1.27)) hide)
     )
@@
       (effects (font (size 1.27 1.27)) hide)
     )
-    (property "LCSC" "" (id 4) (at 121.92 101.6 0)
+    (property "LCSC" "C22939" (id 4) (at 121.92 101.6 0)
       (effects (font (size 1.27 1.27)) hide)
     )
@@
       (effects (font (size 1.27 1.27)) hide)
     )
-    (property "LCSC" "" (id 4) (at 129.54 76.2 0)
+    (property "LCSC" "C25744" (id 4) (at 129.54 76.2 0)
       (effects (font (size 1.27 1.27)) hide)
     )
@@
       (effects (font (size 1.27 1.27)) hide)
     )
-    (property "LCSC" "" (id 4) (at 129.54 114.3 0)
+    (property "LCSC" "C25744" (id 4) (at 129.54 114.3 0)
       (effects (font (size 1.27 1.27)) hide)
     )
@@
       (effects (font (size 1.27 1.27)) hide)
     )
-    (property "LCSC" "" (id 4) (at 68.58 132.08 0)
+    (property "LCSC" "C25744" (id 4) (at 68.58 132.08 0)
       (effects (font (size 1.27 1.27)) hide)
     )
@@
       (effects (font (size 1.27 1.27)) hide)
     )
-    (property "LCSC" "C465729" (id 4) (at 218.44 152.4 0)
+    (property "LCSC" "C15849" (id 4) (at 218.44 152.4 0)
       (effects (font (size 1.27 1.27)) hide)
     )
@@
       (effects (font (size 1.27 1.27)) hide)
     )
-    (property "LCSC" "" (id 4) (at 251.46 106.68 0)
+    (property "LCSC" "C23164" (id 4) (at 251.46 106.68 0)
       (effects (font (size 1.27 1.27)) hide)
     )
@@
       (effects (font (size 1.27 1.27)) hide)
     )
-    (property "LCSC" "" (id 4) (at 251.46 68.58 0)
+    (property "LCSC" "C25744" (id 4) (at 251.46 68.58 0)
       (effects (font (size 1.27 1.27)) hide)
     )
@@
       (effects (font (size 1.27 1.27)) hide)
     )
-    (property "LCSC" "" (id 4) (at 259.08 119.38 0)
+    (property "LCSC" "C25744" (id 4) (at 259.08 119.38 0)
       (effects (font (size 1.27 1.27)) hide)
     )
@@
       (effects (font (size 1.27 1.27)) hide)
     )
-    (property "LCSC" "" (id 4) (at 259.08 81.28 0)
+    (property "LCSC" "C25744" (id 4) (at 259.08 81.28 0)
       (effects (font (size 1.27 1.27)) hide)
     )
@@
       (effects (font (size 1.27 1.27)) hide)
     )
-    (property "LCSC" "" (id 4) (at 172.72 175.26 0)
+    (property "LCSC" "C25744" (id 4) (at 172.72 175.26 0)
       (effects (font (size 1.27 1.27)) hide)
     )
@@
       (effects (font (size 1.27 1.27)) hide)
     )
-    (property "LCSC" "" (id 4) (at 185.42 175.26 0)
-      (effects (font (size 1.27 1.27)) hide)
-    )
+    (property "LCSC" "C25744" (id 4) (at 185.42 175.26 0)
+      (effects (font (size 1.27 1.27)) hide)
+    )

Commit message: Rev E: isolated flyback aux supply, VREF+ back to 3.3 V, 1 oz re-layout
- New isolated aux flyback (sheet iso_pwr): UC3843B U20 from +10V_P, FDN86246 Q11,
  PA3855.006NLT EP13 T2, SS110 D9 -> isolated +10 V; secondary regulation TL431 U22 +
  EL357N opto U21 into COMP; RCD clamp D8/R116/C94; 2 A primary limit (R114)
- Secondary rails from the flyback, not VBUS: +10 V -> U4 10->5 V -> U5 TLV75533 3.3 V;
  MCU, CAN and drivers up before the LLC starts
- U12 -> CA-IS3742LW (data only); REF3030 U19 removed, VREF+ = +3V3A (3.3 V full scale)
- PCB re-placed / re-routed for 1 oz outer / 0.5 oz inner: power pours on F.Cu, In1 solid
  ground planes, gate loops as tight HO/HS pairs, 1.7 mm power-via pitch, per-pad GND vias
  in the MCU area; copper loss ~0.5 W at 50 W (03_calculations/copper_check.txt)
- DRC (JLC rules) 0 errors / 0 unconnected; netlist 148 nets / 284 parts 0 errors;
  isolation bands clear; BOM / JLC BOM+CPL / Gerbers / PDFs / design notes / READMEs updated
- Scripts: 04_scripts/pcb5 (placement, pours, routing, floods, island vias, silk),
  03_calculations/flyback_aux.py, copper_check.py

Co-Authored-By: Claude Opus 5.5 <noreply@anthropic.com>
Claude-Session: https://claude.ai/code/session_01A35wrnwFKLPSaRSxxHs471
Parts:
- C69: LCSC (none) -> C15849
- R67, R74: LCSC (none) -> C25744
- R69: LCSC C25744 -> C23164
- U11: LCSC C15849 -> C465729
Changed lines of the file:
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@@
   (title_block
     (title "LLC isolation stage - half-bridge, PQ2620, synchronous rectifier")
-    (date "2026-10-18")
-    (rev "D")
+    (date "2026-10-19")
+    (rev "E")
     (comment 1 "DCDC LLC + 4SBB, 12-48 V in, 1.5-48 V / 5 A out, STM32G474")
     (comment 2 "Sheet 2: LLC isolation stage - half-bridge, PQ2620, synchronous rectifier")
@@
       (effects (font (size 1.27 1.27)) hide)
     )
-    (property "LCSC" "" (id 4) (at 76.2 132.08 0)
+    (property "LCSC" "C25744" (id 4) (at 76.2 132.08 0)
       (effects (font (size 1.27 1.27)) hide)
     )
@@
       (effects (font (size 1.27 1.27)) hide)
     )
-    (property "LCSC" "C15849" (id 4) (at 218.44 152.4 0)
+    (property "LCSC" "C465729" (id 4) (at 218.44 152.4 0)
       (effects (font (size 1.27 1.27)) hide)
     )
@@
       (effects (font (size 1.27 1.27)) hide)
     )
-    (property "LCSC" "" (id 4) (at 241.3 175.26 0)
+    (property "LCSC" "C15849" (id 4) (at 241.3 175.26 0)
       (effects (font (size 1.27 1.27)) hide)
     )
@@
       (effects (font (size 1.27 1.27)) hide)
     )
-    (property "LCSC" "C25744" (id 4) (at 251.46 68.58 0)
+    (property "LCSC" "C23164" (id 4) (at 251.46 68.58 0)
       (effects (font (size 1.27 1.27)) hide)
     )
@@
       (effects (font (size 1.27 1.27)) hide)
     )
-    (property "LCSC" "" (id 4) (at 198.12 175.26 0)
-      (effects (font (size 1.27 1.27)) hide)
-    )
+    (property "LCSC" "C25744" (id 4) (at 198.12 175.26 0)
+      (effects (font (size 1.27 1.27)) hide)
+    )

Commit message: Rev E BOM: in-stock LCSC first source for every part; 2nd/3rd sources checked
- First sources swapped (same footprints, layout unchanged): U1 STM32G474RBT3,
  Q2/Q3/Q5/Q6 NCEP068N10G, 10k 0402 FOJAN, 100n 0402 merged onto C307331,
  1u 0402 CCTC, R62/R63/R89/R82, FB1 Murata BLM18KG601SN1D, L2/L3 cjiang
  FNR5040S470MT, C82 KEMET C0G (was X7R), RS1 Milliohm HoJLR2512, SS110 MDD
- LCSC part numbers for the hand-soldered headers (J1-J5, J7, JP1)
- Schematic and PCB fields, BOM, JLC BOM/CPL, PDFs and design notes regenerated;
  netlist check 0 errors, DRC unchanged
- BOM_sourcing_revE.xlsx: live LCSC stock 2026-10-20, 2nd/3rd sources checked
  for pinout / land pattern / ratings, PCB reserve options for T2 and U9

Co-Authored-By: Claude Opus 5.5 <noreply@anthropic.com>
Claude-Session: https://claude.ai/code/session_01A35wrnwFKLPSaRSxxHs471
Parts:
- J1: LCSC (none) -> C441204
- Q5, Q6: value NCEP0160AG -> NCEP068N10G; LCSC C503012 -> C503061; MPN NCEP0160AG -> NCEP068N10G
- R62, R63: LCSC C22939 -> C2907006
- R64, R65, R66, R67, R70, R71, R72, R73, R74: LCSC C25744 -> C2906861
Changed lines of the file:
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@@
       (effects (font (size 1.27 1.27)) hide)
     )
-    (property "LCSC" "" (id 4) (at 25.4 63.5 0)
+    (property "LCSC" "C441204" (id 4) (at 25.4 63.5 0)
       (effects (font (size 1.27 1.27)) hide)
     )
@@
       (effects (font (size 1.27 1.27)))
     )
-    (property "Value" "NCEP0160AG" (id 1) (at 135.572 59.09 0)
+    (property "Value" "NCEP068N10G" (id 1) (at 135.572 59.09 0)
       (effects (font (size 1.27 1.27)))
     )
@@
       (effects (font (size 1.27 1.27)) hide)
     )
-    (property "LCSC" "C503012" (id 4) (at 139.7 63.5 0)
-      (effects (font (size 1.27 1.27)) hide)
-    )
-    (property "MPN" "NCEP0160AG" (id 5) (at 139.7 63.5 0)
+    (property "LCSC" "C503061" (id 4) (at 139.7 63.5 0)
+      (effects (font (size 1.27 1.27)) hide)
+    )
+    (property "MPN" "NCEP068N10G" (id 5) (at 139.7 63.5 0)
       (effects (font (size 1.27 1.27)) hide)
     )
@@
       (effects (font (size 1.27 1.27)))
     )
-    (property "Value" "NCEP0160AG" (id 1) (at 135.572 97.19 0)
+    (property "Value" "NCEP068N10G" (id 1) (at 135.572 97.19 0)
       (effects (font (size 1.27 1.27)))
     )
@@
       (effects (font (size 1.27 1.27)) hide)
     )
-    (property "LCSC" "C503012" (id 4) (at 139.7 101.6 0)
-      (effects (font (size 1.27 1.27)) hide)
-    )
-    (property "MPN" "NCEP0160AG" (id 5) (at 139.7 101.6 0)
+    (property "LCSC" "C503061" (id 4) (at 139.7 101.6 0)
+      (effects (font (size 1.27 1.27)) hide)
+    )
+    (property "MPN" "NCEP068N10G" (id 5) (at 139.7 101.6 0)
       (effects (font (size 1.27 1.27)) hide)
     )
@@
       (effects (font (size 1.27 1.27)) hide)
     )
-    (property "LCSC" "C22939" (id 4) (at 121.92 63.5 0)
+    (property "LCSC" "C2907006" (id 4) (at 121.92 63.5 0)
       (effects (font (size 1.27 1.27)) hide)
     )
@@
       (effects (font (size 1.27 1.27)) hide)
     )
-    (property "LCSC" "C22939" (id 4) (at 121.92 101.6 0)
+    (property "LCSC" "C2907006" (id 4) (at 121.92 101.6 0)
       (effects (font (size 1.27 1.27)) hide)
     )
@@
       (effects (font (size 1.27 1.27)) hide)
     )
-    (property "LCSC" "C25744" (id 4) (at 129.54 76.2 0)
+    (property "LCSC" "C2906861" (id 4) (at 129.54 76.2 0)
       (effects (font (size 1.27 1.27)) hide)
     )
@@
       (effects (font (size 1.27 1.27)) hide)
     )
-    (property "LCSC" "C25744" (id 4) (at 129.54 114.3 0)
+    (property "LCSC" "C2906861" (id 4) (at 129.54 114.3 0)
       (effects (font (size 1.27 1.27)) hide)
     )
@@
       (effects (font (size 1.27 1.27)) hide)
     )
-    (property "LCSC" "C25744" (id 4) (at 68.58 132.08 0)
+    (property "LCSC" "C2906861" (id 4) (at 68.58 132.08 0)
       (effects (font (size 1.27 1.27)) hide)
     )
@@
       (effects (font (size 1.27 1.27)) hide)
     )
-    (property "LCSC" "C25744" (id 4) (at 76.2 132.08 0)
+    (property "LCSC" "C2906861" (id 4) (at 76.2 132.08 0)
       (effects (font (size 1.27 1.27)) hide)
     )
@@
       (effects (font (size 1.27 1.27)) hide)
     )
-    (property "LCSC" "C25744" (id 4) (at 259.08 119.38 0)
+    (property "LCSC" "C2906861" (id 4) (at 259.08 119.38 0)
       (effects (font (size 1.27 1.27)) hide)
     )
@@
       (effects (font (size 1.27 1.27)) hide)
     )
-    (property "LCSC" "C25744" (id 4) (at 259.08 81.28 0)
+    (property "LCSC" "C2906861" (id 4) (at 259.08 81.28 0)
       (effects (font (size 1.27 1.27)) hide)
     )
@@
       (effects (font (size 1.27 1.27)) hide)
     )
-    (property "LCSC" "C25744" (id 4) (at 172.72 175.26 0)
+    (property "LCSC" "C2906861" (id 4) (at 172.72 175.26 0)
       (effects (font (size 1.27 1.27)) hide)
     )
@@
       (effects (font (size 1.27 1.27)) hide)
     )
-    (property "LCSC" "C25744" (id 4) (at 185.42 175.26 0)
+    (property "LCSC" "C2906861" (id 4) (at 185.42 175.26 0)
       (effects (font (size 1.27 1.27)) hide)
     )
@@
       (effects (font (size 1.27 1.27)) hide)
     )
-    (property "LCSC" "C25744" (id 4) (at 198.12 175.26 0)
-      (effects (font (size 1.27 1.27)) hide)
-    )
+    (property "LCSC" "C2906861" (id 4) (at 198.12 175.26 0)
+      (effects (font (size 1.27 1.27)) hide)
+    )
