File: 01_hardware/kicad_project/iso_pwr.kicad_sch (KiCad schematic)
At the start: 31 parts, among them Q11 FDN86246, T2 PA3855.006NLT, U20 UC3843BVD1R2G, U21 EL357N(B), U22 TL431AIDBZR

Commit message: Rev E BOM: in-stock LCSC first source for every part; 2nd/3rd sources checked
- First sources swapped (same footprints, layout unchanged): U1 STM32G474RBT3,
  Q2/Q3/Q5/Q6 NCEP068N10G, 10k 0402 FOJAN, 100n 0402 merged onto C307331,
  1u 0402 CCTC, R62/R63/R89/R82, FB1 Murata BLM18KG601SN1D, L2/L3 cjiang
  FNR5040S470MT, C82 KEMET C0G (was X7R), RS1 Milliohm HoJLR2512, SS110 MDD
- LCSC part numbers for the hand-soldered headers (J1-J5, J7, JP1)
- Schematic and PCB fields, BOM, JLC BOM/CPL, PDFs and design notes regenerated;
  netlist check 0 errors, DRC unchanged
- BOM_sourcing_revE.xlsx: live LCSC stock 2026-10-20, 2nd/3rd sources checked
  for pinout / land pattern / ratings, PCB reserve options for T2 and U9

Co-Authored-By: Claude Opus 5.5 <noreply@anthropic.com>
Claude-Session: https://claude.ai/code/session_01A35wrnwFKLPSaRSxxHs471
Parts:
- C90, C99: LCSC C1525 -> C307331
- D8, D9: LCSC C224219 -> C2482
- R111, R113, R120: LCSC C25744 -> C2906861
Changed lines of the file:
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@@
       (effects (font (size 1.27 1.27)) hide)
     )
-    (property "LCSC" "C1525" (id 4) (at 68.58 125.73 0)
+    (property "LCSC" "C307331" (id 4) (at 68.58 125.73 0)
       (effects (font (size 1.27 1.27)) hide)
     )
@@
       (effects (font (size 1.27 1.27)) hide)
     )
-    (property "LCSC" "C25744" (id 4) (at 76.2 127.0 0)
+    (property "LCSC" "C2906861" (id 4) (at 76.2 127.0 0)
       (effects (font (size 1.27 1.27)) hide)
     )
@@
       (effects (font (size 1.27 1.27)) hide)
     )
-    (property "LCSC" "C25744" (id 4) (at 132.08 121.92 0)
+    (property "LCSC" "C2906861" (id 4) (at 132.08 121.92 0)
       (effects (font (size 1.27 1.27)) hide)
     )
@@
       (effects (font (size 1.27 1.27)) hide)
     )
-    (property "LCSC" "C224219" (id 4) (at 172.72 55.88 0)
+    (property "LCSC" "C2482" (id 4) (at 172.72 55.88 0)
       (effects (font (size 1.27 1.27)) hide)
     )
@@
       (effects (font (size 1.27 1.27)) hide)
     )
-    (property "LCSC" "C224219" (id 4) (at 238.76 68.58 0)
+    (property "LCSC" "C2482" (id 4) (at 238.76 68.58 0)
       (effects (font (size 1.27 1.27)) hide)
     )
@@
       (effects (font (size 1.27 1.27)) hide)
     )
-    (property "LCSC" "C25744" (id 4) (at 292.1 166.37 0)
+    (property "LCSC" "C2906861" (id 4) (at 292.1 166.37 0)
       (effects (font (size 1.27 1.27)) hide)
     )
@@
       (effects (font (size 1.27 1.27)) hide)
     )
-    (property "LCSC" "C1525" (id 4) (at 271.78 166.37 0)
-      (effects (font (size 1.27 1.27)) hide)
-    )
+    (property "LCSC" "C307331" (id 4) (at 271.78 166.37 0)
+      (effects (font (size 1.27 1.27)) hide)
+    )
